File: Projects/Client Name/DF_ESC/Design/rev01/rev01_1/DF_ESC_rev01_1/OVERVIEW.kicad_sch (KiCad schematic)
At the start: 0 parts

Commit message: Update 19-01-2024 primera
cambiar y añadir numeracion de sheets
Other:
- note added: "[1] - OVERVIEW"
Changed lines of the file:
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@@
     (comment 4 "Ivan Mendez")
   )
+  (text "[1] - OVERVIEW" (at 99.06 27.94 0)
+    (effects (font (size 8 8) (thickness 1.6) bold) (justify left bottom))
+  )
 )
