File: Projects/Client Name/DF_ESC/Design/rev01/rev01_1/DF_ESC_rev01_1/INPUT PROTECTION.kicad_sch (KiCad schematic)
At the start: 0 parts

Commit message: Update 2024-02-28_2
Input Proteccion Done
Parts:
- added C1, C?: 100n, symbol Device:C
- added C? (x2): LKMI2501K821MF, DF_ESC_Footprint_Library:CAP-TH_BD18.0-P7.50-D1.2-SIDE, symbol DF_ESC_Symbol_Library:LKMI2501K821MF
- added CN?: XT60PW-M, DF_ESC_Footprint_Library:CONN-TH_XT60PW-M, symbol DF_ESC_Symbol_Library:XT60PW-M
- added D?: LED_G, symbol Device:LED
- added D?: SMAJ60CA, Diode_SMD:D_SMA, symbol Diode:SMAJ60CA
- added R1, R?: 2k2, symbol Device:R
- added R? (x2): 39k, symbol Device:R
- added TH2: Thermistor_NTC, symbol Device:Thermistor_NTC
- added U1: XH-2PWBPZ, footprint:CONN-SMD_XH-2PWBPZ, symbol XH-2PWBPZ:XH-2PWBPZ
Connections:
- new net: D?.2 (A), R?.2
- new net +3V3: C1.1, R1.1
- new net +VDC: C?.1, C?.1, CN?.2 (+), D?.2 (A2), R?.1, R?.1
- new net ADC_TEMP: R1.2, TH2.1, U1.2
- new net AN_IN: C?.1, R?.1, R?.2
- new net GND: C1.2, C?.2, C?.2, C?.2, CN?.1 (-), D?.1 (A1), D?.1 (K), R?.2, TH2.2, U1.1
- no-connect marks 0 -> 4
Other:
- note added: "BULK CAPACITANCE"
- note added: "CAN BE USED AS SENSOR ON THE BOARD OR SENSOR ON THE MOTOR"
- note added: "ESD SURGE PROTECTION"
- note added: "FEEDBACK MCU"
- note added: "LED POWER-ON INDICATOR"
- note added: "NTC THERMISTOR"
- note added: "PLACE AS CLOSE AS POSSIBLE TO THE CONNECTOR"
- note added: "PLACE AS CLOSE AS POSSIBLE TO THE DRIVER MOSFETS"
- note added: "POWER INPUT => MAX +60V"
- note added: "VOLTAGE_DIVIDER"
- note added: "WHEN: VDC = 60V => AN_IN = 3V204"
- note added: "[2] - INPUT PROTECTION"
- note removed: "0-60V"
- note removed: "CAN"
- note removed: "COM"
- note removed: "HALL/ENCODER"
- note removed: "MCU"
- note removed: "MOSFET_DRIVER"
- note removed: "MOSFETs"
- note removed: "MOTOR"
- note removed: "SERVO"
- note removed: "TEMP_SENSOR"
- note removed: "USB"
- note removed: "V_SUPPLY"
- note removed: "[2] - BLOCK DIAGRAM"

Commit message: update 2024-02-29
CAN Page DONE
Parts:
- removed CN?: XT60PW-M, DF_ESC_Footprint_Library:CONN-TH_XT60PW-M, symbol DF_ESC_Symbol_Library:XT60PW-M
- removed D?: SMAJ60CA, Diode_SMD:D_SMA, symbol Diode:SMAJ60CA
- added CN1: XT60PW-M, DF_ESC_Footprint_Library:CONN-TH_XT60PW-M, symbol DF_ESC_Symbol_Library:XT60PW-M
- added D4: SMAJ60CA, Diode_SMD:D_SMA_Handsoldering, symbol Diode:SMAJ60CA
Connections:
- net +VDC: now also CN1.2 (+), D4.2 (A2)
- net GND: now also CN1.1 (-), D4.1 (A1)
Changed lines of the file:
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@@
-    )
-  )
-  (symbol (lib_id "DF_ESC_Symbol_Library:XT60PW-M") (at 70.104 85.344 180) (unit 1)
-    (in_bom yes) (on_board yes) (dnp no) (fields_autoplaced)
-    (property "Reference" "CN?" (at 64.262 73.914 0)
-      (effects (font (size 1.27 1.27)) (justify left))
-    )
-    (property "Value" "XT60PW-M" (at 64.262 76.454 0)
-      (effects (font (size 1.27 1.27)) (justify left))
-    )
-    (property "Footprint" "DF_ESC_Footprint_Library:CONN-TH_XT60PW-M" (at 62.484 92.71 0)
-      (effects (font (size 1.27 1.27) italic) hide)
-    )
-    (property "Datasheet" "https://atta.szlcsc.com/upload/public/pdf/source/20180125/C98732_15168617837851301983.pdf" (at 77.216 90.17 0)
-      (effects (font (size 1.27 1.27)) (justify left) hide)
-    )
-    (property "LCSC" "C98732" (at 72.898 94.742 0)
-      (effects (font (size 1.27 1.27)) hide)
-    )
-    (pin "3")
-    (pin "1")
-    (pin "2")
-    (pin "4")
-    (instances
-      (project "DF_ESC_rev01_1"
-        (path "/e63e39d7-6ac0-4ffd-8aa3-1841a4541b55/45b6accf-3fc1-445c-ae1c-ee972cc3cd8b"
-          (reference "CN?") (unit 1)
-        )
-      )
     )
   )
@@
         (path "/e63e39d7-6ac0-4ffd-8aa3-1841a4541b55/45b6accf-3fc1-445c-ae1c-ee972cc3cd8b"
           (reference "#PWR04") (unit 1)
-        )
-      )
-    )
-  )
-  (symbol (lib_id "Diode:SMAJ60CA") (at 93.472 78.232 90) (unit 1)
-    (in_bom yes) (on_board yes) (dnp no) (fields_autoplaced)
-    (property "Reference" "D?" (at 95.504 76.962 90)
-      (effects (font (size 1.27 1.27)) (justify right))
-    )
-    (property "Value" "SMAJ60CA" (at 95.504 79.502 90)
-      (effects (font (size 1.27 1.27)) (justify right))
-    )
-    (property "Footprint" "Diode_SMD:D_SMA" (at 98.552 78.232 0)
-      (effects (font (size 1.27 1.27)) hide)
-    )
-    (property "Datasheet" "https://www.littelfuse.com/media?resourcetype=datasheets&itemid=75e32973-b177-4ee3-a0ff-cedaf1abdb93&filename=smaj-datasheet" (at 93.472 78.232 0)
-      (effects (font (size 1.27 1.27)) hide)
-    )
-    (pin "2")
-    (pin "1")
-    (instances
-      (project "DF_ESC_rev01_1"
-        (path "/e63e39d7-6ac0-4ffd-8aa3-1841a4541b55/45b6accf-3fc1-445c-ae1c-ee972cc3cd8b"
-          (reference "D?") (unit 1)
         )
       )
@@
     )
   )
+  (symbol (lib_id "Diode:SMAJ60CA") (at 93.472 78.232 90) (unit 1)
+    (in_bom yes) (on_board yes) (dnp no) (fields_autoplaced)
+    (property "Reference" "D4" (at 96.012 76.962 90)
+      (effects (font (size 1.27 1.27)) (justify right))
+    )
+    (property "Value" "SMAJ60CA" (at 96.012 79.502 90)
+      (effects (font (size 1.27 1.27)) (justify right))
+    )
+    (property "Footprint" "Diode_SMD:D_SMA_Handsoldering" (at 98.552 78.232 0)
+      (effects (font (size 1.27 1.27)) hide)
+    )
+    (property "Datasheet" "https://www.littelfuse.com/media?resourcetype=datasheets&itemid=75e32973-b177-4ee3-a0ff-cedaf1abdb93&filename=smaj-datasheet" (at 93.472 78.232 0)
+      (effects (font (size 1.27 1.27)) hide)
+    )
+    (pin "1")
+    (pin "2")
+    (instances
+      (project "DF_ESC_rev01_1"
+        (path "/e63e39d7-6ac0-4ffd-8aa3-1841a4541b55/45b6accf-3fc1-445c-ae1c-ee972cc3cd8b"
+          (reference "D4") (unit 1)
+        )
+      )
+    )
+  )
   (symbol (lib_id "power:+VDC") (at 237.744 65.786 0) (unit 1)
     (in_bom yes) (on_board yes) (dnp no) (fields_autoplaced)
@@
         )
       )
+    )
+  )
+  (symbol (lib_id "DF_ESC_Symbol_Library:XT60PW-M") (at 70.104 85.344 180) (unit 1)
+    (in_bom yes) (on_board yes) (dnp no) (fields_autoplaced)
+    (property "Reference" "CN1" (at 63.5 73.914 0)
+      (effects (font (size 1.27 1.27)) (justify left))
+    )
+    (property "Value" "XT60PW-M" (at 63.5 76.454 0)
+      (effects (font (size 1.27 1.27)) (justify left))
+    )
+    (property "Footprint" "DF_ESC_Footprint_Library:CONN-TH_XT60PW-M" (at 62.484 92.71 0)
+      (effects (font (size 1.27 1.27) italic) hide)
+    )
+    (property "Datasheet" "https://atta.szlcsc.com/upload/public/pdf/source/20180125/C98732_15168617837851301983.pdf" (at 77.216 90.17 0)
+      (effects (font (size 1.27 1.27)) (justify left) hide)
+    )
+    (property "LCSC" "C98732" (at 72.898 94.742 0)
+      (effects (font (size 1.27 1.27)) hide)
+    )
+    (pin "1")
+    (pin "4")
+    (pin "2")
+    (pin "3")
+    (instances
+      (project "DF_ESC_rev01_1"
+        (path "/e63e39d7-6ac0-4ffd-8aa3-1841a4541b55/45b6accf-3fc1-445c-ae1c-ee972cc3cd8b"
+          (reference "CN1") (unit 1)
+        )
+      )

Commit message: Update 2024-02-03
Schematic finish but DRC CHEK Errors
Parts:
- C1, C2: renamed from C?; footprint DF_ESC_Footprint_Library:CAP-TH_BD18.0-P7.50-D1.2-SIDE -> DF_ESC_Footprint_Library_Casa:CAP-TH_BD18.0-P7.50-D1.2-SIDE
- C3: renamed from C1; footprint (none) -> Capacitor_SMD:C_0603_1608Metric_Pad1.08x0.95mm_HandSolder
- C4: renamed from C?; footprint (none) -> Capacitor_SMD:C_0603_1608Metric_Pad1.08x0.95mm_HandSolder
- D2: renamed from D?; footprint (none) -> LED_SMD:LED_1206_3216Metric_Pad1.42x1.75mm_HandSolder
- J1: renamed from CN1; footprint DF_ESC_Footprint_Library:CONN-TH_XT60PW-M -> DF_ESC_Footprint_Library_Casa:CONN-TH_XT60PW-M
- R1: footprint (none) -> Resistor_SMD:R_0603_1608Metric_Pad0.98x0.95mm_HandSolder
- R2, R3, R4: renamed from R?; footprint (none) -> Resistor_SMD:R_0603_1608Metric_Pad0.98x0.95mm_HandSolder
- TH1: renamed from TH2; footprint (none) -> Resistor_SMD:R_0603_1608Metric_Pad0.98x0.95mm_HandSolder
- renumbered D4 to D1
