File: Projects/Client Name/DF_ESC/Design/rev01/rev01_1/DF_ESC_rev01_1/INPUT PROTECTION.kicad_sch (KiCad schematic)
At the start: 13 parts, among them J1 XT60PW-M, U1 XH-2PWBPZ

Commit message: update 2024-03-12_1
Parts:
- C1, C2: footprint DF_ESC_Footprint_Library_Casa:CAP-TH_BD18.0-P7.50-D1.2-SIDE -> DF_ESC_Footprint_Library:CAP-TH_BD18.0-P7.50-D1.2-SIDE
- J1: footprint DF_ESC_Footprint_Library_Casa:CONN-TH_XT60PW-M -> DF_ESC_Footprint_Library:CONN-TH_XT60PW-M
- U1: footprint footprint:CONN-SMD_XH-2PWBPZ -> conector_XH2PWBPZ:CONN-SMD_XH-2PWBPZ
- renumbered C4 to C3, C3 to C4, R4 to R1, R1 to R4
