File: Projects/Client Name/DF_ESC/Design/rev01/rev01_1/DF_ESC_rev01_1/INPUT PROTECTION.kicad_sch (KiCad schematic)
At the start: 13 parts, among them J1 XT60PW-M, U1 XH-2PWBPZ

Commit message: Update 2024-03-13_2
Version final para posicionar PCB
Parts:
- U1: footprint footprint:CONN-SMD_XH-2PWBPZ -> DF_ESC_Footprint_Library:CONN-SMD_XH-2PWBPZ
Changed lines of the file:
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@@
 			)
 		)
-		(property "Footprint" "footprint:CONN-SMD_XH-2PWBPZ"
+		(property "Footprint" "DF_ESC_Footprint_Library:CONN-SMD_XH-2PWBPZ"
 			(at 110.49 140.97 0)
 			(effects

Commit message: update 17-03-2024_2
Parts:
- C1: footprint DF_ESC_Footprint_Library_Casa:CAP-TH_BD18.0-P7.50-D1.2-SIDE -> DF_ESC_Footprint_Library:CAP-TH_BD18.0-P7.50-D1.2-SIDE
Changed lines of the file:
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@@
 			)
 		)
-		(property "Footprint" "DF_ESC_Footprint_Library_Casa:CAP-TH_BD18.0-P7.50-D1.2-SIDE"
+		(property "Footprint" "DF_ESC_Footprint_Library:CAP-TH_BD18.0-P7.50-D1.2-SIDE"
 			(at 135.636 79.502 0)
 			(effects

Commit message: update 20240427
Mejora de layout cero errores, solo falta añadir algunas reseñas en el silkscreen
Parts:
- U1: footprint DF_ESC_Footprint_Library:CONN-SMD_XH-2PWBPZ -> footprint:CONN-SMD_XH-2PWBPZ
Changed lines of the file:
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@@
 			)
 		)
-		(property "Footprint" "DF_ESC_Footprint_Library:CONN-SMD_XH-2PWBPZ"
+		(property "Footprint" "footprint:CONN-SMD_XH-2PWBPZ"
 			(at 110.49 140.97 0)
 			(effects
