File: Projects/Client Name/DF_ESC/Design/rev01/rev01_1/DF_ESC_rev01_1/CAN.kicad_sch (KiCad schematic)
At the start: 0 parts

Commit message: Update 14-01-2023
Block diagram
Other:
- title: Title of the project -> DF_ESC_rev01_1
Changed lines of the file:
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@@
   (paper "A4")
   (title_block
-    (title "Title of the project")
+    (title "DF_ESC_rev01_1")
     (date "2024-01-14")
-    (rev "rev01")
+    (rev "rev01_1")
     (company "Ivan Mendez IMA Design")
     (comment 3 "i.mendezalon@hotmail.com")
     (comment 4 "Ivan Mendez")
   )
-  (sheet_instances
-    (path "/" (page "1"))
-  )
 )

Commit message: Update 19-01-2024 primera
cambiar y añadir numeracion de sheets
Other:
- note added: "[4] - BUS CAN"
Changed lines of the file:
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@@
     (comment 4 "Ivan Mendez")
   )
+  (text "[4] - BUS CAN" (at 92.71 29.21 0)
+    (effects (font (size 8 8) (thickness 1.6) bold) (justify left bottom))
+  )
 )

Commit message: update 2024-02-29
CAN Page DONE
Parts:
- added C4, C5, C8: 51p, symbol Device:C
- added R4: 120R, symbol Device:R
- added R5, R6, R7: 10R, symbol Device:R
- added U3: S4B-XH-SM4-TB-(LF)(SN), DF_ESC_Footprint_Library:CONN-SMD_S4B-XH-SM4-TB-LF-SN, symbol DF_ESC_Symbol_Library:S4B-XH-SM4-TB-(LF)(SN)
- added U4: ESDCAN24-2BLY, CAN_TVS:SOT-23-3_L3.0-W1.7-P0.95-LS2.9-BR, symbol ESDCAN24-2BLY:ESDCAN24-2BLY
- added U5: 744227S, DF_ESC_Footprint_Library:FILTER-SMD_4P-L9.2-W6.0-P2.54-TL, symbol DF_ESC_Symbol_Library:744227S
- added U6: SN65HVD230, Package_SO:SOIC-8_3.9x4.9mm_P1.27mm, symbol Interface_CAN_LIN:SN65HVD230
Connections:
- new net: R7.2, U6.8 (Rs)
- new net +3V3: C5.1, U6.3 (VCC)
- new net +5V: U3.4
- new net CAN_N: U5.4, U6.6 (CANL)
- new net CAN_P: U5.3, U6.7 (CANH)
- new net CAN_TX: U6.1 (D), U6.4 (R)
- new net C_CAN_N: C8.1, R4.2, R6.1, U3.2, U4.2
- new net C_CAN_P: C4.2, R4.1, R5.1, U3.3, U4.1
- new net GND: C4.1, C5.2, C8.2, R7.1, U3.1, U4.3, U6.2 (GND)
- new net R_CAN_N: R6.2, U5.1
- new net R_CAN_P: R5.2, U5.2
- no-connect marks 0 -> 3
Other:
- note added: "BYPASS PLACA AS CLOSE AS POSSIBLE TO THE IC"
- note added: "CAN_H Y CAN_L TO BE ROUTED AS DIFFERENTIAL PAIR"
- note added: "LOGIC DIAGRAM"
- note added: "MODE SELECTION RESISTOR SLEW RATE OF-15 V/µs MORE INFO IN DATASHEET"

Commit message: Update 2024-02-03
Schematic finish but DRC CHEK Errors
Parts:
- C52: renamed from C4; footprint (none) -> Capacitor_SMD:C_0603_1608Metric_Pad1.08x0.95mm_HandSolder
- C53: renamed from C8; footprint (none) -> Capacitor_SMD:C_0603_1608Metric_Pad1.08x0.95mm_HandSolder
- C54: renamed from C5; footprint (none) -> Capacitor_SMD:C_0603_1608Metric_Pad1.08x0.95mm_HandSolder
- R44: renamed from R4; footprint (none) -> Resistor_SMD:R_0603_1608Metric_Pad0.98x0.95mm_HandSolder
- R45: renamed from R5; footprint (none) -> Resistor_SMD:R_0603_1608Metric_Pad0.98x0.95mm_HandSolder
- R46: renamed from R6; footprint (none) -> Resistor_SMD:R_0603_1608Metric_Pad0.98x0.95mm_HandSolder
- R47: renamed from R7; footprint (none) -> Resistor_SMD:R_0603_1608Metric_Pad0.98x0.95mm_HandSolder
- U6: renamed from U3; footprint DF_ESC_Footprint_Library:CONN-SMD_S4B-XH-SM4-TB-LF-SN -> DF_ESC_Footprint_Library_Casa:CONN-SMD_S4B-XH-SM4-TB-LF-SN
- U8: renamed from U5; footprint DF_ESC_Footprint_Library:FILTER-SMD_4P-L9.2-W6.0-P2.54-TL -> DF_ESC_Footprint_Library_Casa:FILTER-SMD_4P-L9.2-W6.0-P2.54-TL
- renumbered U4 to U7, U6 to U9
Other:
- note added: "[7] - BUS CAN"
- note removed: "[4] - BUS CAN"

Commit message: Update 2024-03-03
ERC 0 Errors. Update PCB from schematics prepare to going on
Connections:
- net CAN_TX: no longer U9.4 (R)
- new net CAN_RX: U9.4 (R)
Changed lines of the file:
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@@
     (effects (font (size 1.27 1.27)) (justify left bottom))
   )
-  (label "CAN_TX" (at 239.776 92.71 0) (fields_autoplaced)
+  (label "CAN_RX" (at 239.776 92.71 0) (fields_autoplaced)
     (effects (font (size 1.27 1.27)) (justify left bottom))
   )
-  (global_label "CAN_TX" (shape input) (at 249.936 92.71 0) (fields_autoplaced)
+  (global_label "CAN_RX" (shape input) (at 249.936 92.71 0) (fields_autoplaced)
     (effects (font (size 1.27 1.27)) (justify left))
-    (property "Intersheetrefs" "${INTERSHEET_REFS}" (at 259.8501 92.71 0)
+    (property "Intersheetrefs" "${INTERSHEET_REFS}" (at 260.1525 92.71 0)
       (effects (font (size 1.27 1.27)) (justify left) hide)
     )

Commit message: Update 2024-03-03_2
Parts:
- renumbered C52 to C50, C53 to C51, C54 to C52, R44 to R41, R45 to R42, R46 to R43, R47 to R44, U6 to U5, U7 to U6, U8 to U7, U9 to U8
