File: Projects/Client Name/DF_ESC/Design/rev01/rev01_1/DF_ESC_rev01_1/CAN.kicad_sch (KiCad schematic)
At the start: 11 parts, among them U5 S4B-XH-SM4-TB-(LF)(SN), U6 ESDCAN24-2BLY, U7 744227S, U8 SN65HVD230

Commit message: update 2024-03-12_1
Parts:
- U5: renamed from U7; footprint DF_ESC_Footprint_Library_Casa:FILTER-SMD_4P-L9.2-W6.0-P2.54-TL -> DF_ESC_Footprint_Library:FILTER-SMD_4P-L9.2-W6.0-P2.54-TL
- U8: renamed from U5; footprint DF_ESC_Footprint_Library_Casa:CONN-SMD_S4B-XH-SM4-TB-LF-SN -> DF_ESC_Footprint_Library:CONN-SMD_S4B-XH-SM4-TB-LF-SN
- renumbered C52 to C51, C51 to C52, R42 to R41, R41 to R42, U8 to U7
