File: Projects/Client Name/DF_ESC/Design/rev01/rev01_1/DF_ESC_rev01_1/CAN.kicad_sch (KiCad schematic)
At the start: 11 parts, among them U5 S4B-XH-SM4-TB-(LF)(SN), U6 ESDCAN24-2BLY, U7 744227S, U8 SN65HVD230

Commit message: Update 20240416
Lesson 16 finished
Connections:
- net C_CAN_N: now also U6.1; no longer U6.2
- net C_CAN_P: now also U6.2; no longer U6.1
Other:
- moved on the sheet: U6
Changed lines of the file:
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@@
+	)
+	(junction
+		(at 129.54 106.68)
+		(diameter 0)
+		(color 0 0 0 0)
+	)
+	(junction
+		(at 86.36 81.28)
+		(diameter 0)
+		(color 0 0 0 0)
+	)
+	(junction
+		(at 218.44 69.85)
+		(diameter 0)
+		(color 0 0 0 0)
 	)
 	(junction
@@
 	)
 	(junction
-		(at 129.54 106.68)
-		(diameter 0)
-		(color 0 0 0 0)
-	)
-	(junction
-		(at 218.44 69.85)
-		(diameter 0)
-		(color 0 0 0 0)
-	)
-	(junction
-		(at 86.36 81.28)
-		(diameter 0)
-		(color 0 0 0 0)
-	)
-	(junction
 		(at 129.54 81.28)
 		(diameter 0)
@@
 	(wire
 		(pts
-			(xy 86.36 95.25) (xy 86.36 106.68)
+			(xy 86.36 93.98) (xy 86.36 106.68)
 		)
 		(stroke
@@
 	(wire
 		(pts
-			(xy 73.66 81.28) (xy 86.36 81.28)
+			(xy 142.24 55.88) (xy 142.24 63.5)
+		)
+		(stroke
+			(width 0)
+			(type default)
+		)
+	)
+	(wire
+		(pts
+			(xy 166.37 97.79) (xy 176.53 97.79)
 		)
 		(stroke
@@
 	(wire
 		(pts
-			(xy 142.24 55.88) (xy 142.24 63.5)
-		)
-		(stroke
-			(width 0)
-			(type default)
-		)
-	)
-	(wire
-		(pts
-			(xy 166.37 97.79) (xy 176.53 97.79)
+			(xy 86.36 81.28) (xy 129.54 81.28)
 		)
 		(stroke
@@
 	(wire
 		(pts
+			(xy 100.33 91.44) (xy 104.14 91.44)
+		)
+		(stroke
+			(width 0)
+			(type default)
+		)
+	)
+	(wire
+		(pts
 			(xy 199.39 92.71) (xy 208.28 92.71)
 		)
@@
 	(wire
 		(pts
-			(xy 104.14 92.71) (xy 104.14 96.52)
+			(xy 86.36 81.28) (xy 86.36 88.9)
+		)
+		(stroke
+			(width 0)
+			(type default)
+		)
+	)
+	(wire
+		(pts
+			(xy 104.14 91.44) (xy 104.14 96.52)
 		)
 		(stroke
@@
 	(wire
 		(pts
-			(xy 228.6 90.17) (xy 250.19 90.17)
-		)
-		(stroke
-			(width 0)
-			(type default)
-		)
-	)
-	(wire
-		(pts
-			(xy 228.6 97.79) (xy 234.95 97.79)
-		)
-		(stroke
-			(width 0)
-			(type default)
-		)
-	)
-	(wire
-		(pts
-			(xy 86.36 81.28) (xy 129.54 81.28)
+			(xy 86.36 106.68) (xy 129.54 106.68)
 		)
 		(stroke
@@
 	(wire
 		(pts
-			(xy 129.54 87.63) (xy 129.54 81.28)
-		)
-		(stroke
-			(width 0)
-			(type default)
-		)
-	)
-	(wire
-		(pts
-			(xy 157.48 106.68) (xy 166.37 106.68)
+			(xy 228.6 90.17) (xy 250.19 90.17)
+		)
+		(stroke
+			(width 0)
+			(type default)
+		)
+	)
+	(wire
+		(pts
+			(xy 228.6 97.79) (xy 234.95 97.79)
+		)
+		(stroke
+			(width 0)
+			(type default)
+		)
+	)
+	(wire
+		(pts
+			(xy 73.66 81.28) (xy 86.36 81.28)
 		)
 		(stroke
@@
 	(wire
 		(pts
-			(xy 199.39 97.79) (xy 199.39 95.25)
+			(xy 129.54 87.63) (xy 129.54 81.28)
+		)
+		(stroke
+			(width 0)
+			(type default)
+		)
+	)
+	(wire
+		(pts
+			(xy 157.48 106.68) (xy 166.37 106.68)
 		)
 		(stroke
@@
 	(wire
 		(pts
-			(xy 194.31 97.79) (xy 199.39 97.79)
+			(xy 199.39 97.79) (xy 199.39 95.25)
 		)
 		(stroke
@@
 		)
 	)
-	(polyline
-		(pts
-			(xy 237.49 73.66) (xy 246.38 73.66)
-		)
-		(stroke
-			(width 0)
-			(type default)
-		)
-	)
-	(wire
-		(pts
-			(xy 135.89 120.65) (xy 135.89 125.73)
-		)
-		(stroke
-			(width 0)
-			(type default)
-		)
-	)
-	(wire
-		(pts
-			(xy 236.22 69.85) (xy 236.22 73.66)
-		)
-		(stroke
-			(width 0)
-			(type default)
-		)
-	)
-	(wire
-		(pts
-			(xy 101.6 92.71) (xy 104.14 92.71)
-		)
-		(stroke
-			(width 0)
-			(type default)
-		)
-	)
-	(wire
-		(pts
-			(xy 194.31 90.17) (xy 199.39 90.17)
+	(wire
+		(pts
+			(xy 194.31 97.79) (xy 199.39 97.79)
 		)
 		(stroke
@@
 		)
 	)
-	(wire
-		(pts
-			(xy 199.39 95.25) (xy 208.28 95.25)
+	(polyline
+		(pts
+			(xy 237.49 73.66) (xy 246.38 73.66)
+		)
+		(stroke
+			(width 0)
+			(type default)
+		)
+	)
+	(wire
+		(pts
+			(xy 135.89 120.65) (xy 135.89 125.73)
+		)
+		(stroke
+			(width 0)
+			(type default)
+		)
+	)
+	(wire
+		(pts
+			(xy 236.22 69.85) (xy 236.22 73.66)
+		)
+		(stroke
+			(width 0)
+			(type default)
+		)
+	)
+	(wire
+		(pts
+			(xy 194.31 90.17) (xy 199.39 90.17)
 		)
 		(stroke
@@
 	(wire
 		(pts
-			(xy 73.66 93.98) (xy 73.66 106.68)
+			(xy 199.39 95.25) (xy 208.28 95.25)
 		)
 		(stroke
@@
 	(wire
 		(pts
-			(xy 73.66 106.68) (xy 86.36 106.68)
+			(xy 73.66 93.98) (xy 73.66 106.68)
 		)
 		(stroke
@@
 	(wire
 		(pts
-			(xy 88.9 90.17) (xy 86.36 90.17)
-		)
-		(stroke
-			(width 0)
-			(type default)
-		)
-	)
-	(wire
-		(pts
-			(xy 86.36 106.68) (xy 129.54 106.68)
+			(xy 87.63 93.98) (xy 86.36 93.98)
+		)
+		(stroke
+			(width 0)
+			(type default)
+		)
+	)
+	(wire
+		(pts
+			(xy 73.66 106.68) (xy 86.36 106.68)
 		)
 		(stroke
@@
 	(wire
 		(pts
-			(xy 86.36 81.28) (xy 86.36 90.17)
-		)
-		(stroke
-			(width 0)
-			(type default)
-		)
-	)
-	(wire
-		(pts
 			(xy 73.66 91.44) (xy 60.96 91.44)
 		)
@@
 	(wire
 		(pts
+			(xy 87.63 88.9) (xy 86.36 88.9)
+		)
+		(stroke
+			(width 0)
+			(type default)
+		)
+	)
+	(wire
+		(pts
 			(xy 63.5 88.9) (xy 63.5 81.28)
 		)
@@
 			(type solid)
 			(color 132 0 0 1)
-		)
-	)
-	(wire
-		(pts
-			(xy 88.9 95.25) (xy 86.36 95.25)
-		)
-		(stroke
-			(width 0)
-			(type default)
 		)
 	)
@@
 	(symbol
 		(lib_id "ESDCAN24-2BLY:ESDCAN24-2BLY")
-		(at 93.98 92.71 270)
+		(at 92.71 91.44 270)
+		(mirror x)
 		(unit 1)
 		(exclude_from_sim no)
@@
 		(fields_autoplaced yes)
 		(property "Reference" "U6"
-			(at 95.25 83.82 90)
+			(at 93.98 100.33 90)
 			(effects
 				(font
@@
 		)
 		(property "Value" "ESDCAN24-2BLY"
-			(at 95.25 86.36 90)
+			(at 93.98 97.79 90)
 			(effects
 				(font
@@
 		)
 		(property "Footprint" "CAN_TVS:SOT-23-3_L3.0-W1.7-P0.95-LS2.9-BR"
-			(at 83.82 92.71 0)
+			(at 82.55 91.44 0)
 			(effects
 				(font
@@
 		)
 		(property "Datasheet" "https://item.szlcsc.com/139341.html"
-			(at 94.107 90.424 0)
+			(at 92.837 93.726 0)
 			(effects
 				(font
@@
 		)
 		(property "Description" ""
-			(at 93.98 92.71 0)
+			(at 92.71 91.44 0)
 			(effects
 				(font
@@
 		)
 		(property "LCSC" "C246766"
-			(at 93.98 92.71 0)
-			(effects
-				(font
+			(at 92.71 91.44 0)
+			(effects
+				(font

Commit message: update 20240427
Mejora de layout cero errores, solo falta añadir algunas reseñas en el silkscreen
Parts:
- U5: footprint DF_ESC_Footprint_Library_Casa:CONN-SMD_S4B-XH-SM4-TB-LF-SN -> DF_ESC_Footprint_Library:CONN-SMD_S4B-XH-SM4-TB-LF-SN
- U7: footprint DF_ESC_Footprint_Library_Casa:FILTER-SMD_4P-L9.2-W6.0-P2.54-TL -> DF_ESC_Footprint_Library:FILTER-SMD_4P-L9.2-W6.0-P2.54-TL
Changed lines of the file:
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@@
 			)
 		)
-		(property "Footprint" "DF_ESC_Footprint_Library_Casa:CONN-SMD_S4B-XH-SM4-TB-LF-SN"
+		(property "Footprint" "DF_ESC_Footprint_Library:CONN-SMD_S4B-XH-SM4-TB-LF-SN"
 			(at 52.07 109.728 0)
 			(effects
@@
 			)
 		)
-		(property "Footprint" "DF_ESC_Footprint_Library_Casa:FILTER-SMD_4P-L9.2-W6.0-P2.54-TL"
+		(property "Footprint" "DF_ESC_Footprint_Library:FILTER-SMD_4P-L9.2-W6.0-P2.54-TL"
 			(at 200.152 86.36 0)
 			(effects
