File: Projects/Client Name/DF_ESC/Design/rev01/rev01_1/DF_ESC_rev01_1/MECHANICAL.kicad_sch (KiCad schematic)
At the start: 0 parts

Commit message: Update 19-01-2024 primera
cambiar y añadir numeracion de sheets
Other:
- note added: "[8] - MECHANICAL kjlkjlkjlk"
Changed lines of the file:
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@@
     (comment 4 "Ivan Mendez")
   )
+  (text "[8] - MECHANICAL kjlkjlkjlk" (at 101.6 27.94 0)
+    (effects (font (size 8 8) bold) (justify left bottom))
+  )
 )

Commit message: Update 2024-02-03
Schematic finish but DRC CHEK Errors
Parts:
- added B_NAME1: BOARD_NAME, symbol DF_ESC_Symbol_Library_Casa:BOARD_NAME
- added H1, H2, H3, H4: MountingHole_Pad, MountingHole:MountingHole_3.2mm_M3_Pad_Via, symbol Mechanical:MountingHole_Pad
- added LOGO1: DF_LOGO, DF_ESC_Footprint_Library:DF_ESC_REV01_1_LOGO, symbol DF_ESC_Symbol_Library_Casa:DF_LOGO
- added LOGO2: DF_LOGO_NO_SLK, DF_ESC_Footprint_Library:DF_LOGO_NO_SLK, symbol DF_ESC_Symbol_Library_Casa:DF_LOGO_NO_SLK
- added M_DATE1: M_DATE, symbol DF_ESC_Symbol_Library_Casa:M_DATE
- added NOTES1: NOTES, symbol DF_ESC_Symbol_Library_Casa:NOTES
- added PCB1: PCB, symbol DF_ESC_Symbol_Library_Casa:PCB
- added QR1: DF_QR_CODE, DF_ESC_Footprint_Library_Casa:DF_QR_CODE, symbol DF_ESC_Symbol_Library_Casa:DF_QR_CODE
- added R63, R64, R65, R66: 0R, Resistor_SMD:R_0603_1608Metric_Pad0.98x0.95mm_HandSolder, symbol Device:R
Connections:
- new net: H3.1, R65.1
- new net: H1.1, R63.1
- new net: H2.1, R64.1
- new net: H4.1, R66.1
- new net GND: R63.2, R64.2, R65.2, R66.2
Other:
- note added: "FIT A ZERO OHM LINK, CAP OR RESISTOR."
- note added: "IMPORTANT!! COMPATIBLE VESC FIRMWARE 5.02 OTHER VERSIONS MIGHT DAMAGE THE HARDWARE!!"
- note added: "LABELS"
- note added: "LOGOS"
- note added: "MODIFICATION FROM VESC. 4.11: - THERMISTOR MOVED TO LOWER LEG OF THE ADC PIN - BOOT PIN PULLED-DOWN TO GND - CHANGED BULK CPACITANCE - CHANGE PHASE SENSE RESISTORS - CHANGED NETS SENSE PHASES TO DIFFERENTIAL PAIRS - INVERTED TX AND RX CONNECTOR PINS"
- note added: "MOUNTING HOLES"
- note added: "PCB"
- note added: "[10] - MECHANICAL"
- note removed: "[8] - MECHANICAL kjlkjlkjlk"

Commit message: Update 2024-03-03_2
Parts:
- renumbered R63 to R60, R64 to R61, R65 to R62, R66 to R63
Changed lines of the file:
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@@
   (symbol (lib_id "Device:R") (at 81.788 138.938 0) (unit 1)
     (in_bom yes) (on_board yes) (dnp no) (fields_autoplaced)
-    (property "Reference" "R65" (at 83.82 137.668 0)
+    (property "Reference" "R62" (at 83.82 137.668 0)
       (effects (font (size 1.27 1.27)) (justify left))
     )
@@
       (project "DF_ESC_rev01_1"
         (path "/e63e39d7-6ac0-4ffd-8aa3-1841a4541b55/9fe517ea-e439-46a0-9c9c-83eb743bbdc0"
-          (reference "R65") (unit 1)
+          (reference "R62") (unit 1)
         )
       )
@@
   (symbol (lib_id "power:GND") (at 83.312 186.944 0) (unit 1)
     (in_bom yes) (on_board yes) (dnp no) (fields_autoplaced)
-    (property "Reference" "#PWR0104" (at 83.312 193.294 0)
+    (property "Reference" "#PWR0103" (at 83.312 193.294 0)
       (effects (font (size 1.27 1.27)) hide)
     )
@@
       (project "DF_ESC_rev01_1"
         (path "/e63e39d7-6ac0-4ffd-8aa3-1841a4541b55/9fe517ea-e439-46a0-9c9c-83eb743bbdc0"
-          (reference "#PWR0104") (unit 1)
+          (reference "#PWR0103") (unit 1)
         )
       )
@@
   (symbol (lib_id "Device:R") (at 20.32 139.446 0) (unit 1)
     (in_bom yes) (on_board yes) (dnp no) (fields_autoplaced)
-    (property "Reference" "R63" (at 22.352 138.176 0)
+    (property "Reference" "R60" (at 22.352 138.176 0)
       (effects (font (size 1.27 1.27)) (justify left))
     )
@@
       (project "DF_ESC_rev01_1"
         (path "/e63e39d7-6ac0-4ffd-8aa3-1841a4541b55/9fe517ea-e439-46a0-9c9c-83eb743bbdc0"
-          (reference "R63") (unit 1)
+          (reference "R60") (unit 1)
         )
       )
@@
   (symbol (lib_id "Device:R") (at 21.082 181.356 0) (unit 1)
     (in_bom yes) (on_board yes) (dnp no) (fields_autoplaced)
-    (property "Reference" "R64" (at 23.114 180.086 0)
+    (property "Reference" "R61" (at 23.114 180.086 0)
       (effects (font (size 1.27 1.27)) (justify left))
     )
@@
       (project "DF_ESC_rev01_1"
         (path "/e63e39d7-6ac0-4ffd-8aa3-1841a4541b55/9fe517ea-e439-46a0-9c9c-83eb743bbdc0"
-          (reference "R64") (unit 1)
+          (reference "R61") (unit 1)
         )
       )
@@
   (symbol (lib_id "power:GND") (at 81.788 145.034 0) (unit 1)
     (in_bom yes) (on_board yes) (dnp no) (fields_autoplaced)
-    (property "Reference" "#PWR0103" (at 81.788 151.384 0)
+    (property "Reference" "#PWR0102" (at 81.788 151.384 0)
       (effects (font (size 1.27 1.27)) hide)
     )
@@
       (project "DF_ESC_rev01_1"
         (path "/e63e39d7-6ac0-4ffd-8aa3-1841a4541b55/9fe517ea-e439-46a0-9c9c-83eb743bbdc0"
-          (reference "#PWR0103") (unit 1)
+          (reference "#PWR0102") (unit 1)
         )
       )
@@
   (symbol (lib_id "power:GND") (at 20.32 145.288 0) (unit 1)
     (in_bom yes) (on_board yes) (dnp no) (fields_autoplaced)
-    (property "Reference" "#PWR0101" (at 20.32 151.638 0)
+    (property "Reference" "#PWR0100" (at 20.32 151.638 0)
       (effects (font (size 1.27 1.27)) hide)
     )
@@
       (project "DF_ESC_rev01_1"
         (path "/e63e39d7-6ac0-4ffd-8aa3-1841a4541b55/9fe517ea-e439-46a0-9c9c-83eb743bbdc0"
-          (reference "#PWR0101") (unit 1)
+          (reference "#PWR0100") (unit 1)
         )
       )
@@
   (symbol (lib_id "Device:R") (at 83.312 180.848 0) (unit 1)
     (in_bom yes) (on_board yes) (dnp no) (fields_autoplaced)
-    (property "Reference" "R66" (at 85.344 179.578 0)
+    (property "Reference" "R63" (at 85.344 179.578 0)
       (effects (font (size 1.27 1.27)) (justify left))
     )
@@
       (project "DF_ESC_rev01_1"
         (path "/e63e39d7-6ac0-4ffd-8aa3-1841a4541b55/9fe517ea-e439-46a0-9c9c-83eb743bbdc0"
-          (reference "R66") (unit 1)
+          (reference "R63") (unit 1)
         )
       )
@@
   (symbol (lib_id "power:GND") (at 21.082 187.198 0) (unit 1)
     (in_bom yes) (on_board yes) (dnp no) (fields_autoplaced)
-    (property "Reference" "#PWR0102" (at 21.082 193.548 0)
+    (property "Reference" "#PWR0101" (at 21.082 193.548 0)
       (effects (font (size 1.27 1.27)) hide)
     )
@@
       (project "DF_ESC_rev01_1"
         (path "/e63e39d7-6ac0-4ffd-8aa3-1841a4541b55/9fe517ea-e439-46a0-9c9c-83eb743bbdc0"
-          (reference "#PWR0102") (unit 1)
-        )
-      )
+          (reference "#PWR0101") (unit 1)
+        )
+      )
