File: Projects/Client Name/DF_ESC/Design/rev01/rev01_1/DF_ESC_rev01_1/MECHANICAL.kicad_sch (KiCad schematic)
At the start: 15 parts

Commit message: update 2024-03-12_1
Parts:
- QR1: footprint DF_ESC_Footprint_Library_Casa:DF_QR_CODE -> DF_ESC_Footprint_Library:DF_QR_CODE
- renumbered H3 to H1, H1 to H2, H4 to H3, H2 to H4, LOGO2 to LOGO1, LOGO1 to LOGO2, R62 to R60, R60 to R61, R63 to R62, R61 to R63
Changed lines of the file:
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@@
   (symbol (lib_id "DF_ESC_Symbol_Library_Casa:DF_LOGO") (at 30.226 54.61 0) (unit 1)
     (in_bom no) (on_board yes) (dnp no)
-    (property "Reference" "LOGO1" (at 25.908 51.308 0)
+    (property "Reference" "LOGO2" (at 25.908 51.308 0)
       (effects (font (size 1.27 1.27)) (justify left))
     )
@@
       (project "DF_ESC_rev01_1"
         (path "/e63e39d7-6ac0-4ffd-8aa3-1841a4541b55/9fe517ea-e439-46a0-9c9c-83eb743bbdc0"
-          (reference "LOGO1") (unit 1)
+          (reference "LOGO2") (unit 1)
         )
       )
@@
   (symbol (lib_id "Device:R") (at 81.28 138.43 0) (unit 1)
     (in_bom yes) (on_board yes) (dnp no) (fields_autoplaced)
-    (property "Reference" "R62" (at 83.312 137.16 0)
+    (property "Reference" "R60" (at 83.312 137.16 0)
       (effects (font (size 1.27 1.27)) (justify left))
     )
@@
       (project "DF_ESC_rev01_1"
         (path "/e63e39d7-6ac0-4ffd-8aa3-1841a4541b55/9fe517ea-e439-46a0-9c9c-83eb743bbdc0"
-          (reference "R62") (unit 1)
+          (reference "R60") (unit 1)
         )
       )
@@
   (symbol (lib_id "Device:R") (at 20.32 139.7 0) (unit 1)
     (in_bom yes) (on_board yes) (dnp no) (fields_autoplaced)
-    (property "Reference" "R60" (at 22.352 138.43 0)
+    (property "Reference" "R61" (at 22.352 138.43 0)
       (effects (font (size 1.27 1.27)) (justify left))
     )
@@
       (project "DF_ESC_rev01_1"
         (path "/e63e39d7-6ac0-4ffd-8aa3-1841a4541b55/9fe517ea-e439-46a0-9c9c-83eb743bbdc0"
-          (reference "R60") (unit 1)
+          (reference "R61") (unit 1)
         )
       )
@@
   (symbol (lib_id "Device:R") (at 21.59 181.61 0) (unit 1)
     (in_bom yes) (on_board yes) (dnp no) (fields_autoplaced)
-    (property "Reference" "R61" (at 23.622 180.34 0)
+    (property "Reference" "R63" (at 23.622 180.34 0)
       (effects (font (size 1.27 1.27)) (justify left))
     )
@@
       (project "DF_ESC_rev01_1"
         (path "/e63e39d7-6ac0-4ffd-8aa3-1841a4541b55/9fe517ea-e439-46a0-9c9c-83eb743bbdc0"
-          (reference "R61") (unit 1)
+          (reference "R63") (unit 1)
         )
       )
@@
   (symbol (lib_id "DF_ESC_Symbol_Library_Casa:DF_LOGO_NO_SLK") (at 52.578 53.594 0) (unit 1)
     (in_bom no) (on_board yes) (dnp no)
-    (property "Reference" "LOGO2" (at 44.196 51.308 0)
+    (property "Reference" "LOGO1" (at 44.196 51.308 0)
       (effects (font (size 1.27 1.27)) (justify left))
     )
@@
       (project "DF_ESC_rev01_1"
         (path "/e63e39d7-6ac0-4ffd-8aa3-1841a4541b55/9fe517ea-e439-46a0-9c9c-83eb743bbdc0"
-          (reference "LOGO2") (unit 1)
+          (reference "LOGO1") (unit 1)
         )
       )
@@
       (effects (font (size 1.27 1.27)) (justify left))
     )
-    (property "Footprint" "DF_ESC_Footprint_Library_Casa:DF_QR_CODE" (at 73.152 64.008 0)
+    (property "Footprint" "DF_ESC_Footprint_Library:DF_QR_CODE" (at 73.152 64.008 0)
       (effects (font (size 1.27 1.27)) hide)
     )
@@
   (symbol (lib_id "power:GND") (at 81.28 144.78 0) (unit 1)
     (in_bom yes) (on_board yes) (dnp no) (fields_autoplaced)
-    (property "Reference" "#PWR0102" (at 81.28 151.13 0)
+    (property "Reference" "#PWR0101" (at 81.28 151.13 0)
       (effects (font (size 1.27 1.27)) hide)
     )
@@
       (project "DF_ESC_rev01_1"
         (path "/e63e39d7-6ac0-4ffd-8aa3-1841a4541b55/9fe517ea-e439-46a0-9c9c-83eb743bbdc0"
-          (reference "#PWR0102") (unit 1)
+          (reference "#PWR0101") (unit 1)
         )
       )
@@
   (symbol (lib_id "Device:R") (at 83.82 180.34 0) (unit 1)
     (in_bom yes) (on_board yes) (dnp no) (fields_autoplaced)
-    (property "Reference" "R63" (at 85.852 179.07 0)
+    (property "Reference" "R62" (at 85.852 179.07 0)
       (effects (font (size 1.27 1.27)) (justify left))
     )
@@
       (project "DF_ESC_rev01_1"
         (path "/e63e39d7-6ac0-4ffd-8aa3-1841a4541b55/9fe517ea-e439-46a0-9c9c-83eb743bbdc0"
-          (reference "R63") (unit 1)
+          (reference "R62") (unit 1)
         )
       )
@@
   (symbol (lib_id "Mechanical:MountingHole_Pad") (at 20.32 130.81 0) (unit 1)
     (in_bom yes) (on_board yes) (dnp no) (fields_autoplaced)
-    (property "Reference" "H1" (at 23.876 128.27 0)
+    (property "Reference" "H2" (at 23.876 128.27 0)
       (effects (font (size 1.27 1.27)) (justify left))
     )
@@
       (project "DF_ESC_rev01_1"
         (path "/e63e39d7-6ac0-4ffd-8aa3-1841a4541b55/9fe517ea-e439-46a0-9c9c-83eb743bbdc0"
+          (reference "H2") (unit 1)
+        )
+      )
+    )
+  )
+  (symbol (lib_id "Mechanical:MountingHole_Pad") (at 81.28 129.54 0) (unit 1)
+    (in_bom yes) (on_board yes) (dnp no) (fields_autoplaced)
+    (property "Reference" "H1" (at 84.836 127 0)
+      (effects (font (size 1.27 1.27)) (justify left))
+    )
+    (property "Value" "MountingHole_Pad" (at 84.836 129.54 0)
+      (effects (font (size 1.27 1.27)) (justify left))
+    )
+    (property "Footprint" "MountingHole:MountingHole_3.2mm_M3_Pad_Via" (at 81.28 129.54 0)
+      (effects (font (size 1.27 1.27)) hide)
+    )
+    (property "Datasheet" "~" (at 81.28 129.54 0)
+      (effects (font (size 1.27 1.27)) hide)
+    )
+    (pin "1")
+    (instances
+      (project "DF_ESC_rev01_1"
+        (path "/e63e39d7-6ac0-4ffd-8aa3-1841a4541b55/9fe517ea-e439-46a0-9c9c-83eb743bbdc0"
           (reference "H1") (unit 1)
         )
@@
     )
   )
-  (symbol (lib_id "Mechanical:MountingHole_Pad") (at 81.28 129.54 0) (unit 1)
-    (in_bom yes) (on_board yes) (dnp no) (fields_autoplaced)
-    (property "Reference" "H3" (at 84.836 127 0)
-      (effects (font (size 1.27 1.27)) (justify left))
-    )
-    (property "Value" "MountingHole_Pad" (at 84.836 129.54 0)
-      (effects (font (size 1.27 1.27)) (justify left))
-    )
-    (property "Footprint" "MountingHole:MountingHole_3.2mm_M3_Pad_Via" (at 81.28 129.54 0)
-      (effects (font (size 1.27 1.27)) hide)
-    )
-    (property "Datasheet" "~" (at 81.28 129.54 0)
+  (symbol (lib_id "Mechanical:MountingHole_Pad") (at 83.82 171.45 0) (unit 1)
+    (in_bom yes) (on_board yes) (dnp no) (fields_autoplaced)
+    (property "Reference" "H3" (at 87.376 168.91 0)
+      (effects (font (size 1.27 1.27)) (justify left))
+    )
+    (property "Value" "MountingHole_Pad" (at 87.376 171.45 0)
+      (effects (font (size 1.27 1.27)) (justify left))
+    )
+    (property "Footprint" "MountingHole:MountingHole_3.2mm_M3_Pad_Via" (at 83.82 171.45 0)
+      (effects (font (size 1.27 1.27)) hide)
+    )
+    (property "Datasheet" "~" (at 83.82 171.45 0)
       (effects (font (size 1.27 1.27)) hide)
     )
@@
     )
   )
-  (symbol (lib_id "Mechanical:MountingHole_Pad") (at 83.82 171.45 0) (unit 1)
-    (in_bom yes) (on_board yes) (dnp no) (fields_autoplaced)
-    (property "Reference" "H4" (at 87.376 168.91 0)
-      (effects (font (size 1.27 1.27)) (justify left))
-    )
-    (property "Value" "MountingHole_Pad" (at 87.376 171.45 0)
-      (effects (font (size 1.27 1.27)) (justify left))
-    )
-    (property "Footprint" "MountingHole:MountingHole_3.2mm_M3_Pad_Via" (at 83.82 171.45 0)
-      (effects (font (size 1.27 1.27)) hide)
-    )
-    (property "Datasheet" "~" (at 83.82 171.45 0)
-      (effects (font (size 1.27 1.27)) hide)
-    )
-    (pin "1")
-    (instances
-      (project "DF_ESC_rev01_1"
-        (path "/e63e39d7-6ac0-4ffd-8aa3-1841a4541b55/9fe517ea-e439-46a0-9c9c-83eb743bbdc0"
-          (reference "H4") (unit 1)
-        )
-      )
-    )
-  )
   (symbol (lib_id "power:GND") (at 21.59 186.69 0) (unit 1)
     (in_bom yes) (on_board yes) (dnp no) (fields_autoplaced)
-    (property "Reference" "#PWR0101" (at 21.59 193.04 0)
+    (property "Reference" "#PWR0102" (at 21.59 193.04 0)
       (effects (font (size 1.27 1.27)) hide)
     )
@@
       (project "DF_ESC_rev01_1"
         (path "/e63e39d7-6ac0-4ffd-8aa3-1841a4541b55/9fe517ea-e439-46a0-9c9c-83eb743bbdc0"
-          (reference "#PWR0101") (unit 1)
+          (reference "#PWR0102") (unit 1)
         )
       )
@@
   (symbol (lib_id "Mechanical:MountingHole_Pad") (at 21.59 172.72 0) (unit 1)
     (in_bom yes) (on_board yes) (dnp no) (fields_autoplaced)
-    (property "Reference" "H2" (at 25.146 170.18 0)
+    (property "Reference" "H4" (at 25.146 170.18 0)
       (effects (font (size 1.27 1.27)) (justify left))
     )
@@
       (project "DF_ESC_rev01_1"
         (path "/e63e39d7-6ac0-4ffd-8aa3-1841a4541b55/9fe517ea-e439-46a0-9c9c-83eb743bbdc0"
-          (reference "H2") (unit 1)
-        )
-      )
+          (reference "H4") (unit 1)
+        )
+      )
