File: Projects/Client Name/DF_ESC/Design/rev01/rev01_1/DF_ESC_rev01_1/MOSFETs.kicad_sch (KiCad schematic)
At the start: 0 parts

Commit message: Update 19-01-2024 primera
cambiar y añadir numeracion de sheets
Other:
- note added: "[6] - MOSFETs"
Changed lines of the file:
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@@
     (comment 4 "Ivan Mendez")
   )
+  (text "[6] - MOSFETs" (at 102.87 30.48 0)
+    (effects (font (size 8 8) bold) (justify left bottom))
+  )
 )

Commit message: Update 12-02-2024_1
Empiece schematic mosfet
Parts:
- added Q1, Q2, Q3, Q4, Q5, Q6: HSBA15810C, HSBA15810C:PQFN-8_L6.0-W5.0-P1.27-LS6.0-BL, symbol Mosfet_HSBA15810C:HSBA15810C
- added R? (x4): 100R, symbol Device:R
- added R? (x3): 39k, symbol Device:R
- added R? (x6): 4R7, symbol Device:R
- added R? (x2): 0R001, symbol Device:R

Commit message: home Santander 24-02-2024
Acabados los mosfets
Parts:
- removed Q1, Q2, Q3, Q4, Q5, Q6: HSBA15810C, HSBA15810C:PQFN-8_L6.0-W5.0-P1.27-LS6.0-BL, symbol Mosfet_HSBA15810C:HSBA15810C
- removed R? (x4): 100R, symbol Device:R
- removed R? (x3): 39k, symbol Device:R
- removed R? (x6): 4R7, symbol Device:R
- removed R? (x2): 0R001, symbol Device:R
- added C? (x2): 2n2, symbol Device:C
- added J1, J2, J3: 7461084, 7461084:WE_7461084, symbol 7461084:7461084
- added NT? (x6): NetTie_2, symbol Device:NetTie_2
- added NT? (x2): ~, symbol Device:NetTie_2
- added Q? (x6): HSBA15810C, DF_ESC_Footprint_Library:PQFN-8_L6.0-W5.0-P1.27-LS6.0-BL, symbol DF_ESC_Symbol_Library:HSBA15810C
- added R? (x6): 4R7, symbol Device:R
- added R? (x3): 39k, symbol Device:R
- added R? (x4): 100R, symbol Device:R
- added R? (x2): 0R001, symbol Device:R
Connections:
- new net +VDC: Q?.5 (D), Q?.5 (D), Q?.5 (D), Q?.6 (D), Q?.6 (D), Q?.6 (D), Q?.7 (D), Q?.7 (D), Q?.7 (D), Q?.8 (D), Q?.8 (D), Q?.8 (D), Q?.9 (D), Q?.9 (D), Q?.9 (D)
- new net GND: NT?.1, NT?.1, NT?.1, R?.1, R?.1, R?.1
- new net H1_LOW: NT?.2, Q?.1 (S), Q?.2 (S), Q?.3 (S)
- new net H1_VS: NT?.2
- new net H2_LOW: NT?.2, Q?.1 (S), Q?.2 (S), Q?.3 (S)
- new net H2_VS: NT?.2
- new net H3_LOW: NT?.2, Q?.1 (S), Q?.2 (S), Q?.3 (S)
- new net H3_VS: NT?.2
- new net M_H1: R?.1
- new net M_H1_RG: Q?.4 (G), R?.2
- new net M_H2: R?.1
- new net M_H2_RG: Q?.4 (G), R?.2
- new net M_H3: R?.1
- new net M_H3_RG: Q?.4 (G), R?.2
- new net M_L1: R?.1
- new net M_L1_RG: Q?.4 (G), R?.2, R?.2
- new net M_L2: R?.1
- new net M_L2_RG: Q?.4 (G), R?.2, R?.2
- new net M_L3: R?.1
- new net M_L3_RG: Q?.4 (G), R?.2, R?.2
- new net PHASE_1: J1.1, J1.2 (1), J1.3 (1), J1.4 (1), J1.5 (1), J1.6 (1), J1.7 (1), J1.8 (1), NT?.1, Q?.1 (S), Q?.2 (S), Q?.3 (S), Q?.5 (D), Q?.6 (D), Q?.7 (D), Q?.8 (D), Q?.9 (D)
- new net PHASE_2: J2.1, J2.2 (1), J2.3 (1), J2.4 (1), J2.5 (1), J2.6 (1), J2.7 (1), J2.8 (1), NT?.1, Q?.1 (S), Q?.2 (S), Q?.3 (S), Q?.5 (D), Q?.6 (D), Q?.7 (D), Q?.8 (D), Q?.9 (D)
- new net PHASE_3: J3.1, J3.2 (1), J3.3 (1), J3.4 (1), J3.5 (1), J3.6 (1), J3.7 (1), J3.8 (1), NT?.1, Q?.1 (S), Q?.2 (S), Q?.3 (S), Q?.5 (D), Q?.6 (D), Q?.7 (D), Q?.8 (D), Q?.9 (D)
- new net S1_N: C?.1, R?.1
- new net S1_P: C?.2, R?.1
- new net S2_N: C?.1, R?.1
- new net S2_P: C?.2, R?.1
- new net SH1_N: NT?.1, R?.2, R?.2
- new net SH1_P: NT?.2, R?.1, R?.2
- new net SH2_N: NT?.1, R?.2, R?.2
- new net SH2_P: NT?.2, R?.1, R?.2
Other:
- note added: "Hx_Vx"
- note added: "MCU SENSING FEEDBACK FOR EACH FASE"
- note added: "OUTPUT PHASE 1"
- note added: "OUTPUT PHASE 2"
- note added: "OUTPUT PHASE 3"
- note added: "Q_CONTROL"
- note added: "Q_SOURCES"
- note added: "SENSE 1"
- note added: "SENSE 2"

Commit message: Update 2024-02-28_2
Input Proteccion Done
Parts:
- renumbered J3 to J?, J2 to J?, J1 to J?
Other:
- note added: "PLACE AS CLOSE AS POSSIBLE TO THE BULK CAPACITANCE"
- note added: "ROUTE AS KELVIN CONNECTIONS"
- moved on the sheet: NT?, Q?, R?

Commit message: Update 2024-02-03
Schematic finish but DRC CHEK Errors
Parts:
- C50, C51: renamed from C?; footprint (none) -> Capacitor_SMD:C_0603_1608Metric_Pad1.08x0.95mm_HandSolder
- Q1, Q2, Q3, Q4, Q5, Q6: renamed from Q?; footprint DF_ESC_Footprint_Library:PQFN-8_L6.0-W5.0-P1.27-LS6.0-BL -> DF_ESC_Footprint_Library_Casa:PQFN-8_L6.0-W5.0-P1.27-LS6.0-BL
- R29, R30, R31, R32, R33, R34, R35, R36, R37, R38, R39, R40, R41, R42, R43: renamed from R?; footprint (none) -> Resistor_SMD:R_0603_1608Metric_Pad0.98x0.95mm_HandSolder
- gave numbers to parts that had none: 11

Commit message: Update 2024-03-03_2
Parts:
- renumbered C50 to C48, C51 to C49, J3 to J5, J4 to J6, J5 to J7, R29 to R26, R30 to R27, R31 to R28, R32 to R29, R33 to R30, R34 to R31, R35 to R32, R36 to R33, R37 to R34, R38 to R35, R39 to R36, R40 to R37, R41 to R38, R42 to R39, R43 to R40
