File: Projects/Client Name/DF_ESC/Design/rev01/rev01_1/DF_ESC_rev01_1/MOSFETs.kicad_sch (KiCad schematic)
At the start: 34 parts, among them J5 7461084, J6 7461084, J7 7461084, Q1 HSBA15810C, Q2 HSBA15810C, Q3 HSBA15810C, Q4 HSBA15810C, Q5 HSBA15810C, Q6 HSBA15810C

Commit message: update 2024-03-12_1
Parts:
- removed NT2, NT5, NT8: NetTie_2, symbol Device:NetTie_2
- removed NT3, NT6: ~, symbol Device:NetTie_2
- added NT4, NT5, NT6, NT7, NT8: Net_Tie_PWR, DF_ESC_Footprint_Library:NetTie_SMD_Pad_3.00mm, symbol DF_ESC_Symbol_Library_TNP:Net_Tie_PWR
- NT1: footprint (none) -> NetTie:NetTie-2_SMD_Pad0.5mm
- NT2: renamed from NT4; footprint (none) -> NetTie:NetTie-2_SMD_Pad0.5mm
- NT3: renamed from NT7; footprint (none) -> NetTie:NetTie-2_SMD_Pad0.5mm
- Q1, Q6: footprint DF_ESC_Footprint_Library_Casa:PQFN-8_L6.0-W5.0-P1.27-LS6.0-BL -> DF_ESC_Footprint_Library:PQFN-8_L6.0-W5.0-P1.27-LS6.0-BL
- Q2: renamed from Q3; footprint DF_ESC_Footprint_Library_Casa:PQFN-8_L6.0-W5.0-P1.27-LS6.0-BL -> DF_ESC_Footprint_Library:PQFN-8_L6.0-W5.0-P1.27-LS6.0-BL
- Q3: renamed from Q5; footprint DF_ESC_Footprint_Library_Casa:PQFN-8_L6.0-W5.0-P1.27-LS6.0-BL -> DF_ESC_Footprint_Library:PQFN-8_L6.0-W5.0-P1.27-LS6.0-BL
- Q4: renamed from Q2; footprint DF_ESC_Footprint_Library_Casa:PQFN-8_L6.0-W5.0-P1.27-LS6.0-BL -> DF_ESC_Footprint_Library:PQFN-8_L6.0-W5.0-P1.27-LS6.0-BL
- Q5: renamed from Q4; footprint DF_ESC_Footprint_Library_Casa:PQFN-8_L6.0-W5.0-P1.27-LS6.0-BL -> DF_ESC_Footprint_Library:PQFN-8_L6.0-W5.0-P1.27-LS6.0-BL
- renumbered R27 to R26, R33 to R27, R39 to R28, R26 to R29, R32 to R30, R38 to R31, R30 to R32, R36 to R33, R40 to R34, R28 to R35, R34 to R36, R31 to R37, R37 to R38, R29 to R39, R35 to R40
Connections:
- net GND: now also NT6.1, NT7.1, NT8.1
- net H1_LOW: now also NT4.2
- net H2_LOW: now also NT5.2
- net H3_LOW: now also NT6.2
- net SH1_N: now also NT4.1
- net SH1_P: now also NT7.2
- net SH2_N: now also NT5.1
- net SH2_P: now also NT8.2
