File: Projects/Client Name/DF_ESC/Design/rev01/rev01_1/DF_ESC_rev01_1/FILTERS.kicad_sch (KiCad schematic)
At the start: 0 parts

Commit message: Update 19-01-2024 primera
cambiar y añadir numeracion de sheets
Other:
- note added: "[7] - FILTERS"
Changed lines of the file:
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@@
     (comment 4 "Ivan Mendez")
   )
+  (text "[7] - FILTERS " (at 106.68 29.21 0)
+    (effects (font (size 8 8) bold) (justify left bottom))
+  )
 )

Commit message: Update 2024-02-03
Schematic finish but DRC CHEK Errors
Parts:
- added C55, C56, C57, C58: 4n7, Capacitor_SMD:C_0603_1608Metric_Pad1.08x0.95mm_HandSolder, symbol Device:C
- added C59, C60, C61, C62: 100n, Capacitor_SMD:C_0603_1608Metric_Pad1.08x0.95mm_HandSolder, symbol Device:C
- added R48, R49, R50, R51: 2k2, Resistor_SMD:R_0603_1608Metric_Pad0.98x0.95mm_HandSolder, symbol Device:R
- added R52, R53, R54, R55: 10k, Resistor_SMD:R_0603_1608Metric_Pad0.98x0.95mm_HandSolder, symbol Device:R
- added U10: S6B-XH-SM4-TB(LF)(SN), DF_ESC_Footprint_Library:CONN-SMD_S6B-XH-SM4-TB-LF-SN, symbol DF_ESC_Symbol_Library_Casa:S6B-XH-SM4-TB(LF)(SN)
Connections:
- new net +5V: C59.1, C60.1, C61.1, C62.1, R48.1, R49.1, R50.1, R51.1, U10.1
- new net GND: C55.2, C56.2, C57.2, C58.2, C59.2, C60.2, C61.2, C62.2, U10.6
- new net HALL_1_IN: C55.1, R48.2, R52.1, U10.3
- new net HALL_1_OUT: R52.2
- new net HALL_2_IN: C56.1, R49.2, R53.1, U10.4
- new net HALL_2_OUT: R53.2
- new net HALL_3_IN: C57.1, R50.2, R54.1, U10.5
- new net HALL_3_OUT: R54.2
- new net HALL_4_IN: C58.1, R51.2, R55.1
- new net HALL_4_OUT: R55.2
- new net TEMP_IN: U10.2
- no-connect marks 0 -> 2
Other:
- note added: "CONN_01_06"
- note added: "HALL ENCODER"
- note added: "HALL ENCODER OUTPUT"
- note added: "HALL_1_FILTER"
- note added: "HALL_2_FILTER"
- note added: "HALL_3_FILTER"
- note added: "HALL_4_FILTER"
- note added: "INPUT"
- note added: "TO MCU"
- note added: "[8] - FILTERS"
- note removed: "[7] - FILTERS"

Commit message: Update 2024-03-03
ERC 0 Errors. Update PCB from schematics prepare to going on
Connections:
- net HALL_4_IN is gone; now on net TEMP_IN: C58.1, R51.2, R55.1
- net HALL_4_OUT is gone; now on net TEMP_MOTOR: R55.2
- net +5V: now also U10.6; no longer U10.1
- net GND: now also U10.1; no longer U10.6
- net HALL_1_IN: now also U10.4; no longer U10.3
- net HALL_2_IN: now also U10.3; no longer U10.4
- net HALL_3_IN: now also U10.2; no longer U10.5
- net TEMP_IN: now also U10.5; no longer U10.2
Other:
- moved on the sheet: U10
Changed lines of the file:
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@@
     (effects (font (size 1.27 1.27)) (justify right bottom))
   )
-  (label "HALL_4_OUT" (at 152.4 179.07 0) (fields_autoplaced)
+  (label "TEMP_MOTOR" (at 152.4 179.07 0) (fields_autoplaced)
     (effects (font (size 1.27 1.27)) (justify left bottom))
   )
@@
     (effects (font (size 1.27 1.27)) (justify left bottom))
   )
-  (label "HALL_4_IN" (at 87.63 179.07 180) (fields_autoplaced)
+  (label "TEMP_IN" (at 87.63 179.07 180) (fields_autoplaced)
     (effects (font (size 1.27 1.27)) (justify right bottom))
   )
@@
     )
   )
-  (symbol (lib_id "DF_ESC_Symbol_Library_Casa:S6B-XH-SM4-TB(LF)(SN)") (at 36.83 90.17 0) (mirror y) (unit 1)
-    (in_bom yes) (on_board yes) (dnp no) (fields_autoplaced)
-    (property "Reference" "U10" (at 27.94 87.63 0)
-      (effects (font (size 1.27 1.27)) (justify left))
-    )
-    (property "Value" "S6B-XH-SM4-TB(LF)(SN)" (at 27.94 90.17 0)
+  (symbol (lib_id "DF_ESC_Symbol_Library_Casa:S6B-XH-SM4-TB(LF)(SN)") (at 36.83 87.63 180) (unit 1)
+    (in_bom yes) (on_board yes) (dnp no)
+    (property "Reference" "U10" (at 27.94 90.17 0)
+      (effects (font (size 1.27 1.27)) (justify left))
+    )
+    (property "Value" "S6B-XH-SM4-TB(LF)(SN)" (at 27.94 87.63 0)
       (effects (font (size 1.27 1.27)) (justify left) hide)
     )
-    (property "Footprint" "DF_ESC_Footprint_Library:CONN-SMD_S6B-XH-SM4-TB-LF-SN" (at 36.83 100.33 0)
+    (property "Footprint" "DF_ESC_Footprint_Library:CONN-SMD_S6B-XH-SM4-TB-LF-SN" (at 36.83 77.47 0)
       (effects (font (size 1.27 1.27) italic) hide)
     )
-    (property "Datasheet" "https://atta.szlcsc.com/upload/public/pdf/source/20180829/C191914_CF07A40963D925B3D86855552B2C46AC.pdf" (at 39.116 90.043 0)
+    (property "Datasheet" "https://atta.szlcsc.com/upload/public/pdf/source/20180829/C191914_CF07A40963D925B3D86855552B2C46AC.pdf" (at 39.116 87.757 0)
       (effects (font (size 1.27 1.27)) (justify left) hide)
     )
-    (property "LCSC" "C191914" (at 36.83 90.17 0)
-      (effects (font (size 1.27 1.27)) hide)
-    )
+    (property "LCSC" "C191914" (at 36.83 87.63 0)
+      (effects (font (size 1.27 1.27)) hide)
+    )

Commit message: Update 2024-03-03_2
Parts:
- renumbered C55 to C53, C56 to C54, C57 to C55, C58 to C56, C59 to C57, C60 to C58, C61 to C59, C62 to C60, R48 to R45, R49 to R46, R50 to R47, R51 to R48, R52 to R49, R53 to R50, R54 to R51, R55 to R52, U10 to U9

Commit message: update 2024-03-12_1
Parts:
- renumbered C57 to C53, C53 to C54, C58 to C55, C54 to C56, C59 to C57, C55 to C58, C60 to C59, C56 to C60, R49 to R46, R46 to R47, R50 to R48, R47 to R49, R51 to R50, R48 to R51
