File: Projects/Client Name/DF_ESC/Design/rev01/rev01_1/DF_ESC_rev01_1/FILTERS.kicad_sch (KiCad schematic)
At the start: 17 parts, among them U9 S6B-XH-SM4-TB(LF)(SN)

Commit message: Update 20240416
Lesson 16 finished
Connections:
- net +5V: no longer C57.1, C58.1, C59.1, C60.1, R45.1, R46.1, R47.1, R48.1
- new net +3V3: C57.1, C58.1, C59.1, C60.1, R45.1, R46.1, R47.1, R48.1
Other:
- note added: "HALL_1 FILTER"
- note added: "HALL_2 FILTER"
- note added: "HALL_3 FILTER"
- note added: "TEMP_MOTOR FILTER"
- note removed: "HALL_1_FILTER"
- note removed: "HALL_2_FILTER"
- note removed: "HALL_3_FILTER"
- note removed: "HALL_4_FILTER"
