File: Projects/Client Name/DF_ESC/Design/rev01/rev01_1/DF_ESC_rev01_1/STEP DOWN.kicad_sch (KiCad schematic)
At the start: 10 parts, among them U2 AMS1117-3.3

Commit message: update 2024-03-12_1
Parts:
- renumbered C7 to C5, C8 to C6, C5 to C7, C6 to C8, D4 to D3, D5 to D4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
