File: Projects/Client Name/DF_ESC/Design/rev01/rev01_1/DF_ESC_rev01_1/USB.kicad_sch (KiCad schematic)
At the start: 9 parts, among them J8 USB_C_Receptacle_USB2.0, U10 PUSB3AB6Z

Commit message: update 2024-03-12_1
Parts:
- J8: footprint DF_ESC_Footprint_Library_Casa:USB-C_SMD-TYPE-C-31-M-12 -> DF_ESC_Footprint_Library:USB-C_SMD-TYPE-C-31-M-12
- U10: footprint DF_ESC_Footprint_Library_Casa:XSON-7_L2.2-W1.2-P0.50-BL -> DF_ESC_Footprint_Library:XSON-7_L2.2-W1.2-P0.50-BL
- renumbered R55 to R53, R57 to R54, R56 to R55, R58 to R56, R59 to R57, R53 to R58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
