File: Projects/Client Name/DF_ESC/Design/rev01/rev01_1/DF_ESC_rev01_1/DF_ESC_rev01_1.kicad_pcb (KiCad board)
At the start: 2 copper layers, 65 x 56 mm, 4 parts

Commit message: Update DF_ESC_rev01_1.kicad_pcb
Parts:
- added C1: LKMI2501K821MF, DF_ESC_Footprint_Library_Casa:CAP-TH_BD18.0-P7.50-D1.2-SIDE, F.Cu at (7.67, 4.39)
- added C10: 100n, Capacitor_SMD:C_0603_1608Metric_Pad1.08x0.95mm_HandSolder, F.Cu at (1.68, 76.9)
- added C11: 100n, Capacitor_SMD:C_0603_1608Metric_Pad1.08x0.95mm_HandSolder, F.Cu at (1.68, 79.4)
- added C12: 100n, Capacitor_SMD:C_0603_1608Metric_Pad1.08x0.95mm_HandSolder, F.Cu at (1.68, 81.9)
- added C13: C, Capacitor_SMD:C_0603_1608Metric_Pad1.08x0.95mm_HandSolder, F.Cu at (1.68, 84.4)
- added C14: C, Capacitor_SMD:C_0603_1608Metric_Pad1.08x0.95mm_HandSolder, F.Cu at (1.68, 87.0)
- added C15: 100n, Capacitor_SMD:C_0603_1608Metric_Pad1.08x0.95mm_HandSolder, F.Cu at (1.68, 89.5)
- added C16: 100n, Capacitor_SMD:C_0603_1608Metric_Pad1.08x0.95mm_HandSolder, F.Cu at (1.68, 92.0)
- added C17: 100n, Capacitor_SMD:C_0603_1608Metric_Pad1.08x0.95mm_HandSolder, F.Cu at (6.03, 74.4)
- added C18: 2u2, Capacitor_SMD:C_0603_1608Metric_Pad1.08x0.95mm_HandSolder, F.Cu at (6.03, 76.9)
- added C19: 100n, Capacitor_SMD:C_0603_1608Metric_Pad1.08x0.95mm_HandSolder, F.Cu at (6.03, 79.4)
- added C2: LKMI2501K821MF, DF_ESC_Footprint_Library_Casa:CAP-TH_BD18.0-P7.50-D1.2-SIDE, F.Cu at (28.0, 4.39)
- added C20: 2u2, Capacitor_SMD:C_0603_1608Metric_Pad1.08x0.95mm_HandSolder, F.Cu at (6.03, 81.9)
- added C21: 100n, Capacitor_SMD:C_0603_1608Metric_Pad1.08x0.95mm_HandSolder, F.Cu at (6.03, 84.4)
- added C22: 1u, Capacitor_SMD:C_0603_1608Metric_Pad1.08x0.95mm_HandSolder, F.Cu at (6.03, 87.0)
- added C23: 100n, Capacitor_SMD:C_0603_1608Metric_Pad1.08x0.95mm_HandSolder, F.Cu at (6.03, 89.5)
- added C24: 2u2, Capacitor_SMD:C_0603_1608Metric_Pad1.08x0.95mm_HandSolder, F.Cu at (48.7, 26.5)
- added C25: 2u2, Capacitor_SMD:C_0603_1608Metric_Pad1.08x0.95mm_HandSolder, F.Cu at (48.7, 29.0)
- added C26: 10n, Capacitor_SMD:C_0603_1608Metric_Pad1.08x0.95mm_HandSolder, F.Cu at (48.7, 31.6)
- added C27: 2u2, Capacitor_SMD:C_0603_1608Metric_Pad1.08x0.95mm_HandSolder, F.Cu at (48.7, 34.1)
- added C28: 2u2, Capacitor_SMD:C_0603_1608Metric_Pad1.08x0.95mm_HandSolder, F.Cu at (48.7, 36.6)
- added C29: 120p, Capacitor_SMD:C_0603_1608Metric_Pad1.08x0.95mm_HandSolder, F.Cu at (48.7, 39.1)
- added C3: 100n, Capacitor_SMD:C_0603_1608Metric_Pad1.08x0.95mm_HandSolder, F.Cu at (42.3, 0.76)
- added C30: 22n, Capacitor_SMD:C_0603_1608Metric_Pad1.08x0.95mm_HandSolder, F.Cu at (48.7, 41.6)
- added C31: 2u2, Capacitor_SMD:C_0603_1608Metric_Pad1.08x0.95mm_HandSolder, F.Cu at (48.7, 44.1)
- added C32: 100n, Capacitor_SMD:C_0603_1608Metric_Pad1.08x0.95mm_HandSolder, F.Cu at (48.7, 46.6)
- added C33: 100n, Capacitor_SMD:C_0603_1608Metric_Pad1.08x0.95mm_HandSolder, F.Cu at (53.0, 26.5)
- added C34: 100n, Capacitor_SMD:C_0603_1608Metric_Pad1.08x0.95mm_HandSolder, F.Cu at (53.0, 29.0)
- added C35: 100n, Capacitor_SMD:C_0603_1608Metric_Pad1.08x0.95mm_HandSolder, F.Cu at (53.0, 31.6)
- added C36: 1u, Capacitor_SMD:C_0603_1608Metric_Pad1.08x0.95mm_HandSolder, F.Cu at (53.0, 34.1)
- added C37: 1u, Capacitor_SMD:C_0603_1608Metric_Pad1.08x0.95mm_HandSolder, F.Cu at (53.0, 36.6)
- added C38: 1u, Capacitor_SMD:C_0603_1608Metric_Pad1.08x0.95mm_HandSolder, F.Cu at (53.0, 39.1)
- added C39: 100n, Capacitor_SMD:C_0603_1608Metric_Pad1.08x0.95mm_HandSolder, F.Cu at (53.0, 41.6)
- added C4: 100n, Capacitor_SMD:C_0603_1608Metric_Pad1.08x0.95mm_HandSolder, F.Cu at (42.3, 3.27)
- added C40: 1u, Capacitor_SMD:C_0603_1608Metric_Pad1.08x0.95mm_HandSolder, F.Cu at (53.0, 44.1)
- added C41: 10u, Capacitor_SMD:C_0603_1608Metric_Pad1.08x0.95mm_HandSolder, F.Cu at (53.0, 46.6)
- added C42: 100n, Capacitor_SMD:C_0603_1608Metric_Pad1.08x0.95mm_HandSolder, F.Cu at (57.4, 26.5)
- added C43: 10u, Capacitor_SMD:C_0603_1608Metric_Pad1.08x0.95mm_HandSolder, F.Cu at (57.4, 29.0)
- added C44: 1u, Capacitor_SMD:C_0603_1608Metric_Pad1.08x0.95mm_HandSolder, F.Cu at (57.4, 31.6)
- added C45: 10u, Capacitor_SMD:C_0603_1608Metric_Pad1.08x0.95mm_HandSolder, F.Cu at (57.4, 34.1)
- added C46: 100n, Capacitor_SMD:C_0603_1608Metric_Pad1.08x0.95mm_HandSolder, F.Cu at (57.4, 36.6)
- added C47: 1u, Capacitor_SMD:C_0603_1608Metric_Pad1.08x0.95mm_HandSolder, F.Cu at (57.4, 39.1)
- added C48: 2n2, Capacitor_SMD:C_0603_1608Metric_Pad1.08x0.95mm_HandSolder, F.Cu at (48.7, 9.47)
- added C49: 2n2, Capacitor_SMD:C_0603_1608Metric_Pad1.08x0.95mm_HandSolder, F.Cu at (48.7, 12.0)
- added C5: 1u, Capacitor_SMD:C_0603_1608Metric_Pad1.08x0.95mm_HandSolder, F.Cu at (78.7, 26.5)
- added C50: 51p, Capacitor_SMD:C_0603_1608Metric_Pad1.08x0.95mm_HandSolder, F.Cu at (68.4, 51.1)
- added C51: 51p, Capacitor_SMD:C_0603_1608Metric_Pad1.08x0.95mm_HandSolder, F.Cu at (68.4, 53.6)
- added C52: 51p, Capacitor_SMD:C_0603_1608Metric_Pad1.08x0.95mm_HandSolder, F.Cu at (68.4, 56.1)
- added C53: 4n7, Capacitor_SMD:C_0603_1608Metric_Pad1.08x0.95mm_HandSolder, F.Cu at (85.6, 74.0)
- added C54: 4n7, Capacitor_SMD:C_0603_1608Metric_Pad1.08x0.95mm_HandSolder, F.Cu at (85.6, 76.5)
- added C55: 4n7, Capacitor_SMD:C_0603_1608Metric_Pad1.08x0.95mm_HandSolder, F.Cu at (85.6, 79.0)
- added C56: 4n7, Capacitor_SMD:C_0603_1608Metric_Pad1.08x0.95mm_HandSolder, F.Cu at (85.6, 81.6)
- added C57: 100n, Capacitor_SMD:C_0603_1608Metric_Pad1.08x0.95mm_HandSolder, F.Cu at (85.6, 84.1)
- added C58: 100n, Capacitor_SMD:C_0603_1608Metric_Pad1.08x0.95mm_HandSolder, F.Cu at (85.6, 86.6)
- added C59: 100n, Capacitor_SMD:C_0603_1608Metric_Pad1.08x0.95mm_HandSolder, F.Cu at (90.0, 74.0)
- added C6: 1u, Capacitor_SMD:C_0603_1608Metric_Pad1.08x0.95mm_HandSolder, F.Cu at (78.7, 29.0)
- added C60: 100n, Capacitor_SMD:C_0603_1608Metric_Pad1.08x0.95mm_HandSolder, F.Cu at (90.0, 76.5)
- added C7: 1u, Capacitor_SMD:C_0603_1608Metric_Pad1.08x0.95mm_HandSolder, F.Cu at (78.7, 31.6)
- added C8: 1u, Capacitor_SMD:C_0603_1608Metric_Pad1.08x0.95mm_HandSolder, F.Cu at (78.7, 34.1)
- added C9: 10u, Capacitor_SMD:C_0603_1608Metric_Pad1.08x0.95mm_HandSolder, F.Cu at (1.68, 74.4)
- added D1: SMAJ60CA, Diode_SMD:D_SMA_Handsoldering, F.Cu at (23.9, 43.2)
- added D10: BAT60A, Diode_SMD:D_SOD-323, F.Cu at (29.2, 80.5)
- added D11: LED_G, LED_SMD:LED_1206_3216Metric_Pad1.42x1.75mm_HandSolder, F.Cu at (34.3, 78.2)
- added D12: LED_R, LED_SMD:LED_1206_3216Metric_Pad1.42x1.75mm_HandSolder, F.Cu at (34.3, 81.6)
- added D13: BAT60A, Diode_SMD:D_SOD-323, F.Cu at (29.2, 83.5)
- added D14: PMEG6020AELR, Diode_SMD:Nexperia_CFP3_SOD-123W, F.Cu at (66.7, 36.5)
- added D15: BAT60A, Diode_SMD:D_SOD-323, F.Cu at (71.7, 36.3)
- added D2: LED_G, LED_SMD:LED_1206_3216Metric_Pad1.42x1.75mm_HandSolder, F.Cu at (21.9, 47.2)
- added D3: LED_G, LED_SMD:LED_1206_3216Metric_Pad1.42x1.75mm_HandSolder, F.Cu at (83.9, 35.3)
- added D4: BAT60A, Diode_SMD:D_SOD-323, F.Cu at (89.1, 35.1)
- added D5: LED_G, LED_SMD:LED_1206_3216Metric_Pad1.42x1.75mm_HandSolder, F.Cu at (83.9, 38.7)
- added D6: LED, LED_SMD:LED_1206_3216Metric_Pad1.42x1.75mm_HandSolder, F.Cu at (34.3, 74.8)
- added D8: BAT60A, Diode_SMD:D_SOD-323, F.Cu at (29.2, 74.6)
- added D9: SD05_SOD323, Diode_SMD:D_SOD-323, F.Cu at (29.2, 77.6)
- added FB1: FerriteBead, Inductor_SMD:L_0603_1608Metric_Pad1.05x0.95mm_HandSolder, F.Cu at (6.03, 92.0)
- added H1: MountingHole_Pad, MountingHole:MountingHole_3.2mm_M3_Pad_Via, F.Cu at (50.5, 53.8)
- added H2: MountingHole_Pad, MountingHole:MountingHole_3.2mm_M3_Pad_Via, F.Cu at (50.5, 61.8)
- added H3: MountingHole_Pad, MountingHole:MountingHole_3.2mm_M3_Pad_Via, F.Cu at (50.5, 69.7)
- added H4: MountingHole_Pad, MountingHole:MountingHole_3.2mm_M3_Pad_Via, F.Cu at (50.5, 77.7)
- added J1: XT60PW-M, DF_ESC_Footprint_Library_Casa:CONN-TH_XT60PW-M, F.Cu at (9.19, 49.3)
- added J3: S6B-XH-SM4-TB(LF)(SN), DF_ESC_Footprint_Library_Casa:CONN-SMD_S6B-XH-SM4-TB-LF-SN, F.Cu at (10.9, 67.5)
- added J4: XH-3AWB, DF_ESC_Footprint_Library_Casa:CONN-SMD_XH-3AWB, F.Cu at (29.1, 65.0)
- added J8: USB_C_Receptacle_USB2.0, DF_ESC_Footprint_Library_Casa:USB-C_SMD-TYPE-C-31-M-12, F.Cu at (76.0, 77.7)
- added L1: 22u, DF_ESC_Footprint_Library_Casa:IND-SMD_L7.8-W7.8_SDR0805, F.Cu at (69.2, 30.1)
- added Q1: HSBA15810C, DF_ESC_Footprint_Library_Casa:PQFN-8_L6.0-W5.0-P1.27-LS6.0-BL, F.Cu at (49.8, 3.62)
- added Q2: HSBA15810C, DF_ESC_Footprint_Library_Casa:PQFN-8_L6.0-W5.0-P1.27-LS6.0-BL, F.Cu at (56.5, 3.62)
- added Q3: HSBA15810C, DF_ESC_Footprint_Library_Casa:PQFN-8_L6.0-W5.0-P1.27-LS6.0-BL, F.Cu at (63.1, 3.62)
- added Q4: HSBA15810C, DF_ESC_Footprint_Library_Casa:PQFN-8_L6.0-W5.0-P1.27-LS6.0-BL, F.Cu at (69.8, 3.62)
- added Q5: HSBA15810C, DF_ESC_Footprint_Library_Casa:PQFN-8_L6.0-W5.0-P1.27-LS6.0-BL, F.Cu at (76.4, 3.62)
- added Q6: HSBA15810C, DF_ESC_Footprint_Library_Casa:PQFN-8_L6.0-W5.0-P1.27-LS6.0-BL, F.Cu at (83.1, 3.62)
- added QR1: DF_QR_CODE, DF_ESC_Footprint_Library_Casa:DF_QR_CODE, F.Cu at (59.5, 63.9)
- added R1: 2k2, Resistor_SMD:R_0603_1608Metric_Pad0.98x0.95mm_HandSolder, F.Cu at (42.3, 5.78)
- added R10: 1k, Resistor_SMD:R_0603_1608Metric_Pad0.98x0.95mm_HandSolder, F.Cu at (10.4, 81.9)
- added R11: 1k, Resistor_SMD:R_0603_1608Metric_Pad0.98x0.95mm_HandSolder, F.Cu at (10.4, 84.4)
- added R12: 0R, Resistor_SMD:R_0603_1608Metric_Pad0.98x0.95mm_HandSolder, F.Cu at (10.4, 87.0)
- added R13: 2k2, Resistor_SMD:R_0603_1608Metric_Pad0.98x0.95mm_HandSolder, F.Cu at (10.4, 89.5)
- added R14: 16k, Resistor_SMD:R_0603_1608Metric_Pad0.98x0.95mm_HandSolder, F.Cu at (57.4, 41.6)
- added R15: 10k, Resistor_SMD:R_0603_1608Metric_Pad0.98x0.95mm_HandSolder, F.Cu at (57.4, 44.1)
- added R16: 205k, Resistor_SMD:R_0603_1608Metric_Pad0.98x0.95mm_HandSolder, F.Cu at (57.4, 46.6)
- added R17: 1M, Resistor_SMD:R_0603_1608Metric_Pad0.98x0.95mm_HandSolder, F.Cu at (61.7, 26.5)
- added R18: 18k, Resistor_SMD:R_0603_1608Metric_Pad0.98x0.95mm_HandSolder, F.Cu at (61.7, 29.0)
- added R19: 3k3, Resistor_SMD:R_0603_1608Metric_Pad0.98x0.95mm_HandSolder, F.Cu at (61.7, 31.6)
- added R2: 39k, Resistor_SMD:R_0603_1608Metric_Pad0.98x0.95mm_HandSolder, F.Cu at (42.3, 8.29)
- added R20: 18k, Resistor_SMD:R_0603_1608Metric_Pad0.98x0.95mm_HandSolder, F.Cu at (61.7, 34.1)
- added R21: 2k2, Resistor_SMD:R_0603_1608Metric_Pad0.98x0.95mm_HandSolder, F.Cu at (61.7, 36.6)
- added R22: 18k, Resistor_SMD:R_0603_1608Metric_Pad0.98x0.95mm_HandSolder, F.Cu at (61.7, 39.1)
- added R23: 2k2, Resistor_SMD:R_0603_1608Metric_Pad0.98x0.95mm_HandSolder, F.Cu at (61.7, 41.6)
- added R24: 18k, Resistor_SMD:R_0603_1608Metric_Pad0.98x0.95mm_HandSolder, F.Cu at (61.7, 44.1)
- added R25: 2k2, Resistor_SMD:R_0603_1608Metric_Pad0.98x0.95mm_HandSolder, F.Cu at (61.7, 46.6)
- added R26: 4R7, Resistor_SMD:R_0603_1608Metric_Pad0.98x0.95mm_HandSolder, F.Cu at (48.7, 14.5)
- added R27: 4R7, Resistor_SMD:R_0603_1608Metric_Pad0.98x0.95mm_HandSolder, F.Cu at (48.7, 17.0)
- added R28: 100R, Resistor_SMD:R_0603_1608Metric_Pad0.98x0.95mm_HandSolder, F.Cu at (48.7, 19.5)
- added R29: 100R, Resistor_SMD:R_0603_1608Metric_Pad0.98x0.95mm_HandSolder, F.Cu at (48.7, 22.0)
- added R3: 2k2, Resistor_SMD:R_0603_1608Metric_Pad0.98x0.95mm_HandSolder, F.Cu at (42.3, 10.8)
- added R30: 39k, Resistor_SMD:R_0603_1608Metric_Pad0.98x0.95mm_HandSolder, F.Cu at (53.0, 9.47)
- added R31: 0R001, Resistor_SMD:R_0603_1608Metric_Pad0.98x0.95mm_HandSolder, F.Cu at (53.0, 12.0)
- added R32: 4R7, Resistor_SMD:R_0603_1608Metric_Pad0.98x0.95mm_HandSolder, F.Cu at (53.0, 14.5)
- added R33: 4R7, Resistor_SMD:R_0603_1608Metric_Pad0.98x0.95mm_HandSolder, F.Cu at (53.0, 17.0)
- added R34: 100R, Resistor_SMD:R_0603_1608Metric_Pad0.98x0.95mm_HandSolder, F.Cu at (53.0, 19.5)
- added R35: 100R, Resistor_SMD:R_0603_1608Metric_Pad0.98x0.95mm_HandSolder, F.Cu at (53.0, 22.0)
- added R36: 39k, Resistor_SMD:R_0603_1608Metric_Pad0.98x0.95mm_HandSolder, F.Cu at (57.4, 9.47)
- added R37: 0R001, Resistor_SMD:R_0603_1608Metric_Pad0.98x0.95mm_HandSolder, F.Cu at (57.4, 12.0)
- added R38: 4R7, Resistor_SMD:R_0603_1608Metric_Pad0.98x0.95mm_HandSolder, F.Cu at (57.4, 14.5)
- added R39: 4R7, Resistor_SMD:R_0603_1608Metric_Pad0.98x0.95mm_HandSolder, F.Cu at (57.4, 17.0)
- added R4: 39k, Resistor_SMD:R_0603_1608Metric_Pad0.98x0.95mm_HandSolder, F.Cu at (42.3, 13.3)
- added R40: 39k, Resistor_SMD:R_0603_1608Metric_Pad0.98x0.95mm_HandSolder, F.Cu at (57.4, 19.5)
- added R41: 120R, Resistor_SMD:R_0603_1608Metric_Pad0.98x0.95mm_HandSolder, F.Cu at (68.4, 58.7)
- added R42: 10R, Resistor_SMD:R_0603_1608Metric_Pad0.98x0.95mm_HandSolder, F.Cu at (68.4, 61.2)
- added R43: 10R, Resistor_SMD:R_0603_1608Metric_Pad0.98x0.95mm_HandSolder, F.Cu at (68.4, 63.7)
- added R44: 10R, Resistor_SMD:R_0603_1608Metric_Pad0.98x0.95mm_HandSolder, F.Cu at (68.4, 66.2)
- added R45: 2k2, Resistor_SMD:R_0603_1608Metric_Pad0.98x0.95mm_HandSolder, F.Cu at (90.0, 79.0)
- added R46: 2k2, Resistor_SMD:R_0603_1608Metric_Pad0.98x0.95mm_HandSolder, F.Cu at (90.0, 81.6)
- added R47: 2k2, Resistor_SMD:R_0603_1608Metric_Pad0.98x0.95mm_HandSolder, F.Cu at (90.0, 84.1)
- added R48: 2k2, Resistor_SMD:R_0603_1608Metric_Pad0.98x0.95mm_HandSolder, F.Cu at (90.0, 86.6)
- added R49: 10k, Resistor_SMD:R_0603_1608Metric_Pad0.98x0.95mm_HandSolder, F.Cu at (94.3, 74.0)
- added R5: 1k, Resistor_SMD:R_0603_1608Metric_Pad0.98x0.95mm_HandSolder, F.Cu at (78.7, 36.6)
- added R50: 10k, Resistor_SMD:R_0603_1608Metric_Pad0.98x0.95mm_HandSolder, F.Cu at (94.3, 76.5)
- added R51: 10k, Resistor_SMD:R_0603_1608Metric_Pad0.98x0.95mm_HandSolder, F.Cu at (94.3, 79.0)
- added R52: 10k, Resistor_SMD:R_0603_1608Metric_Pad0.98x0.95mm_HandSolder, F.Cu at (94.3, 81.6)
- added R53: 0R, Resistor_SMD:R_0603_1608Metric_Pad0.98x0.95mm_HandSolder, F.Cu at (68.4, 74.0)
- added R54: 0R, Resistor_SMD:R_0603_1608Metric_Pad0.98x0.95mm_HandSolder, F.Cu at (68.4, 76.5)
- added R55: 0R, Resistor_SMD:R_0603_1608Metric_Pad0.98x0.95mm_HandSolder, F.Cu at (68.4, 79.0)
- added R56: 5k1, Resistor_SMD:R_0603_1608Metric_Pad0.98x0.95mm_HandSolder, F.Cu at (68.4, 81.6)
- added R57: 5k1, Resistor_SMD:R_0603_1608Metric_Pad0.98x0.95mm_HandSolder, F.Cu at (68.4, 84.1)
- added R58: 22R, Resistor_SMD:R_0603_1608Metric_Pad0.98x0.95mm_HandSolder, F.Cu at (68.4, 86.6)
- added R59: 22R, Resistor_SMD:R_0603_1608Metric_Pad0.98x0.95mm_HandSolder, F.Cu at (68.4, 89.1)
- added R6: 1k, Resistor_SMD:R_0603_1608Metric_Pad0.98x0.95mm_HandSolder, F.Cu at (78.7, 39.1)
- added R60: 0R, Resistor_SMD:R_0603_1608Metric_Pad0.98x0.95mm_HandSolder, F.Cu at (56.6, 51.1)
- added R61: 0R, Resistor_SMD:R_0603_1608Metric_Pad0.98x0.95mm_HandSolder, F.Cu at (56.6, 53.6)
- added R62: 0R, Resistor_SMD:R_0603_1608Metric_Pad0.98x0.95mm_HandSolder, F.Cu at (56.6, 56.1)
- added R63: 0R, Resistor_SMD:R_0603_1608Metric_Pad0.98x0.95mm_HandSolder, F.Cu at (56.6, 58.7)
- added R7: 1k, Resistor_SMD:R_0603_1608Metric_Pad0.98x0.95mm_HandSolder, F.Cu at (10.4, 74.4)
- added R8: R, Resistor_SMD:R_0603_1608Metric_Pad0.98x0.95mm_HandSolder, F.Cu at (10.4, 76.9)
- added R9: R, Resistor_SMD:R_0603_1608Metric_Pad0.98x0.95mm_HandSolder, F.Cu at (10.4, 79.4)
- added SW1: SW_DIP_x01, DF_ESC_Footprint_Library_Casa:SW-SMD_4P-L5.2-W5.2-P3.70-LS6.4, F.Cu at (31.5, 88.5)
- added TH1: Thermistor_NTC, Resistor_SMD:R_0603_1608Metric_Pad0.98x0.95mm_HandSolder, F.Cu at (42.3, 15.8)
- added U10: PUSB3AB6Z, DF_ESC_Footprint_Library_Casa:XSON-7_L2.2-W1.2-P0.50-BL, F.Cu at (72.5, 83.4)
- added U2: AMS1117-3.3, Package_TO_SOT_SMD:SOT-223-3_TabPin2, F.Cu at (85.8, 29.5)
- added U3: STM32F405RGTx, Package_QFP:LQFP-64_10x10mm_P0.5mm, F.Cu at (19.8, 80.4)
- added U5: S4B-XH-SM4-TB-(LF)(SN), DF_ESC_Footprint_Library_Casa:CONN-SMD_S4B-XH-SM4-TB-LF-SN, F.Cu at (80.4, 58.1)
- added U7: 744227S, DF_ESC_Footprint_Library_Casa:FILTER-SMD_4P-L9.2-W6.0-P2.54-TL, F.Cu at (76.7, 67.0)
- added U8: SN65HVD230, Package_SO:SOIC-8_3.9x4.9mm_P1.27mm, F.Cu at (86.2, 66.7)
- added Y1: Crystal_Small, DF_ESC_Footprint_Library_Casa:CRYSTAL-SMD_L5.0-W3.2, F.Cu at (16.5, 90.1)

Commit message: Update 2024-03-13_2
Version final para posicionar PCB
Parts:
- added D7: PESD3V3U1UA,115, PESD3V3U1UA:SOD-323_L1.7-W1.3-LS2.5-RD, F.Cu at (346.6, 199.0)
- added J2: HX25003-8AWB, DF_ESC_Footprint_Library:CONN-SMD_8P-P2.50_HX25003-8AWB, F.Cu at (358.2, 192.5)
- added J5: 7461084, 7461084:WE_7461084, F.Cu at (321.5, 177.5)
- added J6: 7461084, 7461084:WE_7461084, F.Cu at (321.5, 189.1)
- added J7: 7461084, 7461084:WE_7461084, F.Cu at (321.5, 200.6)
- added LOGO1: DF_LOGO, DF_ESC_Footprint_Library:DF_ESC_REV01_1_LOGO, F.Cu at (361.4, 177.1)
- added LOGO2: DF_LOGO_NO_SLK, DF_ESC_Footprint_Library:DF_LOGO_NO_SLK, F.Cu at (357.5, 179.8)
- added NT1: NetTie_2, NetTie:NetTie-2_SMD_Pad0.5mm, F.Cu at (328.5, 177.5)
- added NT2: Net_Tie_PWR, DF_ESC_Footprint_Library:NetTie_SMD_Pad_3.00mm, F.Cu at (328.8, 174.3)
- added NT3: Net_Tie_PWR, DF_ESC_Footprint_Library:NetTie_SMD_Pad_3.00mm, F.Cu at (331.8, 174.3)
- added NT4: NetTie_2, NetTie:NetTie-2_SMD_Pad0.5mm, F.Cu at (328.5, 179.0)
- added NT5: Net_Tie_PWR, DF_ESC_Footprint_Library:NetTie_SMD_Pad_3.00mm, F.Cu at (334.9, 174.3)
- added NT6: Net_Tie_PWR, DF_ESC_Footprint_Library:NetTie_SMD_Pad_3.00mm, F.Cu at (337.9, 174.3)
- added NT7: NetTie_2, NetTie:NetTie-2_SMD_Pad0.5mm, F.Cu at (328.5, 180.5)
- added NT8: Net_Tie_PWR, DF_ESC_Footprint_Library:NetTie_SMD_Pad_3.00mm, F.Cu at (341.0, 174.3)
- added U1: XH-2PWBPZ, DF_ESC_Footprint_Library:CONN-SMD_XH-2PWBPZ, F.Cu at (321.7, 213.6)
- added U4: DRV8302DCAR, DF_ESC_Footprint_Library:HTSSOP-56_L14.0-W6.1-P0.50-LS8.1-BL-EP, F.Cu at (352.6, 222.8)
- added U6: ESDCAN24-2BLY, CAN_TVS:SOT-23-3_L3.0-W1.7-P0.95-LS2.9-BR, F.Cu at (317.8, 224.5)
- added U9: S6B-XH-SM4-TB(LF)(SN), DF_ESC_Footprint_Library:CONN-SMD_S6B-XH-SM4-TB-LF-SN, F.Cu at (355.9, 210.1)
- moved C1 302.4 mm to (304.6, 61.6)
- moved C10 302.4 mm to (298.7, 134.1)
- moved C11 302.4 mm to (298.7, 136.6)
- moved C12 302.4 mm to (298.7, 139.1)
- moved C13 302.4 mm to (298.7, 141.6)
- moved C14 302.4 mm to (298.7, 144.1)
- moved C15 302.4 mm to (298.7, 146.7)
- moved C16 302.4 mm to (298.7, 149.2)
- moved C17 302.4 mm to (303.0, 131.6)
- moved C18 302.4 mm to (303.0, 134.1)
- moved C19 302.4 mm to (303.0, 136.6)
- moved C2 302.4 mm to (325.0, 61.6)
- moved C20 302.4 mm to (303.0, 139.1)
- moved C21 302.4 mm to (303.0, 141.6)
- moved C22 302.4 mm to (303.0, 144.1)
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
Commit message: update 17-03-2024_1
Parts:
- moved C53 343.2 mm to (41.9, 173.2)
- moved C54 343.2 mm to (41.9, 175.7)
- moved C55 343.2 mm to (41.9, 178.2)
- moved C56 343.2 mm to (41.9, 180.8)
- moved C57 343.2 mm to (41.9, 183.3)
- moved C58 343.2 mm to (41.9, 185.8)
- moved C59 343.2 mm to (46.3, 173.2)
- moved C60 343.2 mm to (46.3, 175.7)
- moved R45 343.2 mm to (46.3, 178.2)
- moved R46 343.2 mm to (46.3, 180.8)
- moved R47 343.2 mm to (46.3, 183.3)
- moved R48 343.2 mm to (46.3, 185.8)
- moved R49 343.2 mm to (50.6, 173.2)
- moved R50 343.2 mm to (50.6, 175.7)
- moved R51 343.2 mm to (50.6, 178.2)
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Other:
- board text added: "CAN"
- board text added: "FILTERS"
- board text added: "INPUT PROTECTION"
- board text added: "MCU"
- board text added: "MECHANICAL"
- board text added: "MOSFET"
- board text added: "MOSFET DRIVER"
- board text added: "STEP DOWN"
- board text added: "USB"

Commit message: update 17-03-2024_2
Parts:
- moved R4 47.8 mm to (77.9, 87.9)
- moved C4 47.5 mm to (56.4, 72.8), turned to -90 degrees
- moved R2 44.7 mm to (51.9, 71.9)
- moved R3 41.9 mm to (54.6, 72.8), turned to -90 degrees
- moved C1 28.8 mm to (47.5, 58.0), turned to 180 degrees
- moved C2 28.8 mm to (67.8, 58.0), turned to 180 degrees
- moved C3 22.6 mm to (66.4, 91.9)
- moved R1 15.8 mm to (66.4, 90.1)
- moved U1 13.5 mm to (68.2, 80.7)
- moved D1 11.8 mm to (48.1, 74.5)
- moved C5 11.2 mm to (109.8, 34.9)
- moved R5 11.2 mm to (109.9, 38.5)
- moved C6 11.0 mm to (109.8, 36.7)
- moved D2 10.5 mm to (77.3, 85.8)
- moved C8 7.68 mm to (105.6, 34.9), turned to 180 degrees
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
Commit message: update 2024-03-28
lesson 13 fineshed
Parts:
- moved D7 162.6 mm to (198.1, 183.0)
- moved SW1 45.6 mm to (41.7, 224.7)
- moved J2 42.2 mm to (57.5, 261.3)
- moved Q2 42.0 mm to (205.3, 64.8), turned to 90 degrees
- moved Q1 39.8 mm to (205.3, 58.9), turned to 90 degrees
- moved R29 37.5 mm to (218.5, 53.8), turned to 90 degrees
- moved R38 36.2 mm to (202.4, 70.8), turned to 90 degrees
- moved R28 35.9 mm to (216.0, 53.8), turned to 90 degrees
- moved J4 35.1 mm to (36.4, 249.9), turned to 90 degrees
- moved R39 34.7 mm to (204.9, 70.8), turned to 90 degrees
- moved R27 34.5 mm to (213.5, 53.8), turned to 90 degrees
- moved R40 33.6 mm to (207.4, 70.8), turned to 90 degrees
- moved R26 33.5 mm to (211.0, 53.8), turned to 90 degrees
- moved R35 32.8 mm to (218.5, 36.5), turned to 90 degrees
- moved NT6 30.1 mm to (193.2, 60.0)
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
Commit message: update 07-04-2024
Parts:
- C1: footprint DF_ESC_Footprint_Library_Casa:CAP-TH_BD18.0-P7.50-D1.2-SIDE -> DF_ESC_Footprint_Library:CAP-TH_BD18.0-P7.50-D1.2-SIDE; moved to B.Cu
- C2, C48, C49, R28, R29, R34, R35: moved to B.Cu
- R31, R37: footprint Resistor_SMD:R_0603_1608Metric_Pad0.98x0.95mm_HandSolder -> DF_ESC_Footprint_Library:RES-SMD_L7.0-W6.7
- moved MH1 289.2 mm to (450.8, 11.1)
- moved MH2 289.2 mm to (508.8, 11.1)
- moved MH3 289.2 mm to (450.8, 60.1)
- moved MH4 289.2 mm to (508.8, 60.1)
- moved J1 232.5 mm to (266.0, 106.3), turned to -90 degrees
- moved D1 230.8 mm to (276.0, 110.9), turned to -90 degrees
- moved C1 230.7 mm to (253.0, 162.7), turned to 90 degrees
- moved C3 224.8 mm to (290.4, 110.5)
- moved R1 224.8 mm to (290.4, 108.7)
- moved TH1 224.8 mm to (292.2, 107.0)
- moved J4 223.8 mm to (205.0, 102.7), turned to 0 degrees
- moved H3 223.6 mm to (278.8, 101.1)
- moved J3 210.0 mm to (228.8, 103.6)
- moved D2 206.1 mm to (281.6, 113.1), turned to -90 degrees
- moved R62 203.4 mm to (278.8, 106.6), turned to -90 degrees
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Other:
- board size 65 x 56 mm -> 100 x 75 mm
- board text added: "COM"
- board text added: "PROG"
- board text added: "SENSORS"
- board text added: "SERVO"
- board text removed: "Extend PCB edge 0.5mm if using SMT header"
- board text removed: "MCU"
- board text removed: "MECHANICAL"
- board text removed: "MOSFET"
- board text removed: "MOSFET DRIVER"
- board text removed: "STEP DOWN"
