File: Projects/Client Name/DF_ESC/Design/rev01/rev01_1/DF_ESC_rev01_1/DF_ESC_rev01_1.kicad_pcb (KiCad board)
At the start: 4 copper layers, 100 x 75 mm, 187 parts, among them J1 XT60PW-M, J2 HX25003-8AWB, J3 S6B-XH-SM4-TB(LF)(SN), J4 XH-3AWB, J5 7461084, J6 7461084, J7 7461084, J8 USB_C_Receptacle_USB2.0, Q1 HSBA15810C, Q2 HSBA15810C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

Commit message: update 20240424_2
Ultimos detalles desde casa
Routing:
- net GND: track 130.3 -> 150.2 mm, vias 83 -> 93
- net /[4] - MCU/NRST: track 35.1 -> 50.5 mm
- net /[9] - USB/+5V_C: track 2.61 -> 14.8 mm, vias 0 -> 2
- net +5V: track 200.5 -> 204.2 mm
- net /[4] - MCU/PH_0: track 3.58 -> 5.99 mm
- net /[4] - MCU/+5V_COM: track 4.52 -> 6.71 mm
- net Net-(U3-VDDA): track 4.59 -> 6.11 mm
- net FAULT: track 25.7 -> 26.6 mm
- net /[4] - MCU/SCK_ADC_EXT: track 24.7 -> 25.5 mm

Commit message: Update DF_ESC_rev01_1.kicad_pcb
Parts:
- added G***: LOGO, LOGO, F.Cu at (255.8, 136.3)
- added G***: LOGO, LOGO, F.Cu at (281.6, 108.0)
- added G***: LOGO, LOGO, F.Cu at (223.1, 126.8)
- added G***: LOGO, LOGO, F.Cu at (242.8, 165.7)
- added G***: LOGO, LOGO, F.Cu at (234.4, 165.6)
- added G***: LOGO, LOGO, F.Cu at (248.4, 122.8)
- added G***: LOGO, LOGO, F.Cu at (238.4, 125.4)
- added G***: LOGO, LOGO, F.Cu at (203.2, 150.7)
- moved QR1 240.3 mm to (295.2, 79.1)
- moved LOGO1 195.1 mm to (261.0, 84.0)
- moved LOGO2 11.3 mm to (116.0, -27.6)
- moved R63 1.27 mm to (274.2, 167.0), turned to -90 degrees
Routing:
- net /[4] - MCU/TX_SDA_NSS: track 43.2 -> 44.5 mm
- net +5V: track 204.2 -> 203.1 mm

Commit message: Update DF_ESC_rev01_1.kicad_pcb
Routing:
- net M_H1: track 57.1 -> 56.0 mm, vias 1 -> 0
- net /[9] - USB/CC2: vias 3 -> 2
Changed lines of the file:
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@@
 		(at 238.366839 125.391123 90)
 		(property "Reference" "G***"
-			(at 0 0 270)
+			(at 0 0 -90)
 			(layer "F.SilkS")
 			(hide yes)
@@
 		)
 		(property "Value" "LOGO"
-			(at 0.75 0 270)
+			(at 0.75 0 -90)
 			(layer "F.SilkS")
 			(hide yes)
@@
 	)
 	(via
-		(at 244.72 102.7985)
-		(size 0.6)
-		(drill 0.3)
-		(layers "F.Cu" "B.Cu")
-		(free yes)
-		(net 66)
-	)
-	(via
 		(at 247.32 102.1985)
 		(size 0.6)
@@
 	)
 	(segment
-		(start 277.131227 117.019975)
-		(end 276.043727 117.019975)
-		(width 0.2)
-		(layer "F.Cu")
-		(net 96)
-	)
-	(segment
 		(start 275.82 116.22)
 		(end 276.043727 116.443727)
@@
 		(net 96)
 	)
-	(via
-		(at 277.131227 117.019975)
-		(size 0.6)
-		(drill 0.3)
-		(layers "F.Cu" "B.Cu")
-		(net 96)
-	)
 	(segment
 		(start 258.82 130.22)
@@
 	)
 	(segment
-		(start 218.502 134.289471)
-		(end 217.32 135.471471)
+		(start 212.02 153.125005)
+		(end 212.02 154.251505)
 		(width 0.2)
 		(layer "F.Cu")
@@
 	)
 	(segment
-		(start 212.02 153.125005)
-		(end 212.02 154.251505)
+		(start 217.32 136.82)
+		(end 217.32 135.471471)
 		(width 0.2)
 		(layer "F.Cu")
@@
 	)
 	(segment
-		(start 218.502 133.013)
-		(end 218.502 134.289471)
+		(start 214.120548 140.037714)
+		(end 214.120548 140.019452)
 		(width 0.2)
 		(layer "F.Cu")
@@
 	(segment
 		(start 217.32 135.471471)
-		(end 217.32 136.82)
+		(end 218.502 134.289471)
 		(width 0.2)
 		(layer "F.Cu")
@@
 	)
 	(segment
-		(start 217.32 136.82)
-		(end 213.92 140.22)
+		(start 214.120548 140.019452)
+		(end 217.32 136.82)
+		(width 0.2)
+		(layer "F.Cu")
+		(net 110)
+	)
+	(segment
+		(start 218.502 134.289471)
+		(end 218.502 133.013)
 		(width 0.2)
 		(layer "F.Cu")
@@
 	)
 	(via
-		(at 213.92 140.22)
+		(at 214.120548 140.037714)
 		(size 0.6)
 		(drill 0.3)
@@
 	)
 	(segment
-		(start 213.92 140.22)
-		(end 213.92 146.72)
+		(start 214.12 146.52)
+		(end 211.02 149.62)
 		(width 0.2)
 		(layer "B.Cu")
@@
 	)
 	(segment
-		(start 213.92 146.72)
-		(end 211.02 149.62)
+		(start 214.120548 140.037714)
+		(end 214.12 140.038262)
+		(width 0.2)
+		(layer "B.Cu")
+		(net 110)
+	)
+	(segment
+		(start 214.12 140.038262)
+		(end 214.12 146.52)
 		(width 0.2)
 		(layer "B.Cu")
@@
 	)
 	(segment
+		(start 211.82 138.42)
+		(end 211.802 138.438)
+		(width 0.2)
+		(layer "F.Cu")
+		(net 111)
+	)
+	(segment
 		(start 212.02 146.92)
 		(end 212.62 147.52)
@@
 	)
 	(segment
-		(start 211.82 138.42)
-		(end 211.802 138.438)
+		(start 211.802 138.438)
+		(end 210.577 138.438)
 		(width 0.2)
 		(layer "F.Cu")
@@
 		(net 111)
 	)
-	(segment
-		(start 210.577 138.438)
-		(end 211.802 138.438)
-		(width 0.2)
-		(layer "F.Cu")
-		(net 111)
-	)
 	(via
 		(at 211.82 138.42)
@@
 	)
 	(segment
-		(start 211.82 138.42)
-		(end 211.82 146.72)
+		(start 211.82 146.72)
+		(end 212.02 146.92)
 		(width 0.2)
 		(layer "B.Cu")
@@
 	)
 	(segment
-		(start 211.82 146.72)
-		(end 212.02 146.92)
+		(start 211.82 138.42)
+		(end 211.82 146.72)
 		(width 0.2)
 		(layer "B.Cu")

Commit message: update 20240425_casa
Parts:
- moved D13 4.00 mm to (236.4, 106.3)
Routing:
- net Net-(D13-A): track 1.96 -> 6.06 mm
- net +3V3: track 289.6 -> 293.2 mm
- net GND: track 150.0 -> 148.8 mm

Commit message: update 20240427
Mejora de layout cero errores, solo falta añadir algunas reseñas en el silkscreen
Parts:
- removed MH1, MH2, MH3, MH4: MountingHole_2.7mm_M2.5, MountingHole:MountingHole_2.7mm_M2.5
- added G***: LOGO, LOGO, F.Cu at (280.3, 148.3)
- added G***: LOGO, LOGO, F.Cu at (255.5, 100.4)
- added G***: LOGO, LOGO, F.Cu at (280.3, 131.3)
- J3: footprint DF_ESC_Footprint_Library_Casa:CONN-SMD_S6B-XH-SM4-TB-LF-SN -> DF_ESC_Footprint_Library:CONN-SMD_S6B-XH-SM4-TB-LF-SN
- J4: footprint DF_ESC_Footprint_Library_Casa:CONN-SMD_XH-3AWB -> DF_ESC_Footprint_Library:CONN-SMD_XH-3AWB
- L1: footprint DF_ESC_Footprint_Library_Casa:IND-SMD_L7.8-W7.8_SDR0805 -> DF_ESC_Footprint_Library:IND-SMD_L7.8-W7.8_SDR0805
- LOGO1, LOGO2, QR1: moved to B.Cu
- Q1, Q2, Q3, Q4, Q5, Q6: footprint DF_ESC_Footprint_Library_Casa:PQFN-8_L6.0-W5.0-P1.27-LS6.0-BL -> DF_ESC_Footprint_Library:PQFN-8_L6.0-W5.0-P1.27-LS6.0-BL
- SW1: footprint DF_ESC_Footprint_Library_Casa:SW-SMD_4P-L5.2-W5.2-P3.70-LS6.4 -> DF_ESC_Footprint_Library:SW-SMD_4P-L5.2-W5.2-P3.70-LS6.4
- U10: footprint DF_ESC_Footprint_Library_Casa:XSON-7_L2.2-W1.2-P0.50-BL -> DF_ESC_Footprint_Library:XSON-7_L2.2-W1.2-P0.50-BL
- U5: footprint DF_ESC_Footprint_Library_Casa:CONN-SMD_S4B-XH-SM4-TB-LF-SN -> DF_ESC_Footprint_Library:CONN-SMD_S4B-XH-SM4-TB-LF-SN
- U7: footprint DF_ESC_Footprint_Library_Casa:FILTER-SMD_4P-L9.2-W6.0-P2.54-TL -> DF_ESC_Footprint_Library:FILTER-SMD_4P-L9.2-W6.0-P2.54-TL
- Y1: footprint DF_ESC_Footprint_Library_Casa:CRYSTAL-SMD_L5.0-W3.2 -> DF_ESC_Footprint_Library:CRYSTAL-SMD_L5.0-W3.2
- moved LOGO2 164.7 mm to (201.0, 113.5), turned to 180 degrees
- moved QR1 91.3 mm to (228.2, 141.1), turned to 180 degrees
- moved LOGO1 58.0 mm to (234.9, 135.8), turned to 180 degrees
- moved G*** 9.11 mm to (235.9, 116.6)
- moved C7 3.37 mm to (241.2, 116.0)
- moved NT4 2.46 mm to (277.4, 147.2)
- moved G*** 1.55 mm to (204.7, 150.6)
- moved G*** 0.77 mm to (282.3, 107.7)
- moved R54 0.76 mm to (239.6, 101.3)
- moved G*** 0.60 mm to (233.8, 165.6)
- moved C1 0.57 mm to (257.2, 163.3)
- moved G*** 0.43 mm to (248.8, 122.8)
- moved R43 0.24 mm to (203.8, 119.1)
- moved C16 0.21 mm to (209.2, 132.8)
- moved R42 0.20 mm to (203.8, 121.2)
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Routing:
- net Net-(J8-SHIELD-PadS1): track 12.8 -> 22.3 mm
- net /[9] - USB/USB-C_P: track 43.4 -> 47.3 mm
- net /[3] - STEP DOWN/+3V3_IC: track 13.5 -> 15.1 mm
- net GND: track 148.8 -> 150.3 mm
- net SENS2: track 75.8 -> 74.6 mm
- net H2_VS: track 39.8 -> 40.9 mm
- net /[9] - USB/USB-C_N: track 47.2 -> 48.4 mm
- net +3V3: track 293.2 -> 294.2 mm
- net H1_LOW: track 40.5 -> 39.7 mm, vias 3 -> 2
Other:
- board text added: "+3V3"
- board text added: "+3V3_COM"
- board text added: "+5V"
- board text added: "CAN_N"
- board text added: "CAN_P"
- board text added: "COMM"
- board text added: "GND"
- board text added: "MISO_ADC_EXT2"
- board text added: "NRST"
- board text added: "REF**"
- board text added: "RX_SCL_MOSI"
- board text added: "SCK_ADC_EXT"
- board text added: "SWCLK"
- board text added: "SWDIO"
- board text added: "TX_SDA_NSS"
- board text removed: "COM"
- board text removed: "FILTERS"
- board text removed: "INPUT PROTECTION"
- board text removed: "SENSORS"

Commit message: update 20240428
Other:
- board text added: "+VCC"
- board text added: "ADC_TEMP"
- board text added: "GREEN"
- board text added: "H1"
- board text added: "H2"
- board text added: "H3"
- board text added: "HALL SENSOR"
- board text added: "RED"
- board text added: "TEMP"
- board text added: "THERMISTOR"
Changed lines of the file:
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@@
+		)
+	)
+	(gr_text "HALL SENSOR"
+		(at 214.52 152.22 0)
+		(layer "F.SilkS")
+		(effects
+			(font
+				(size 0.5 0.5)
+				(thickness 0.125)
+			)
+			(justify left bottom)
 		)
 	)
@@
 		)
 	)
+	(gr_text "ADC_TEMP"
+		(at 202.42 159.72 0)
+		(layer "F.SilkS")
+		(effects
+			(font
+				(size 0.5 0.5)
+				(thickness 0.125)
+			)
+			(justify left bottom)
+		)
+	)
+	(gr_text "GREEN"
+		(at 232.42 162.02 0)
+		(layer "F.SilkS")
+		(effects
+			(font
+				(size 0.5 0.5)
+				(thickness 0.125)
+			)
+			(justify left bottom)
+		)
+	)
 	(gr_text "GND"
 		(at 196.42 148.12 0)
@@
 		)
 	)
+	(gr_text "GND\n"
+		(at 261.52 115.82 0)
+		(layer "F.SilkS")
+		(effects
+			(font
+				(size 0.5 0.5)
+				(thickness 0.125)
+			)
+			(justify left bottom)
+		)
+	)
+	(gr_text "GND"
+		(at 210.12 160.32 0)
+		(layer "F.SilkS")
+		(effects
+			(font
+				(size 0.5 0.5)
+				(thickness 0.125)
+			)
+			(justify left bottom)
+		)
+	)
 	(gr_text "CAN_N"
 		(at 191.62 109.62 0)
@@
 		)
 	)
+	(gr_text "+5V"
+		(at 226.22 160.22 0)
+		(layer "F.SilkS")
+		(effects
+			(font
+				(size 0.5 0.5)
+				(thickness 0.125)
+			)
+			(justify left bottom)
+		)
+	)
 	(gr_text "+3V3_COM"
 		(at 196.42 146.52 0)
@@
 		)
 	)
+	(gr_text "H1"
+		(at 219.62 158.72 0)
+		(layer "F.SilkS")
+		(effects
+			(font
+				(size 0.5 0.5)
+				(thickness 0.125)
+			)
+			(justify left bottom)
+		)
+	)
 	(gr_text "GND"
 		(at 196.32 156.12 0)
+		(layer "F.SilkS")
+		(effects
+			(font
+				(size 0.5 0.5)
+				(thickness 0.125)
+			)
+			(justify left bottom)
+		)
+	)
+	(gr_text "H2"
+		(at 217.12 158.72 0)
 		(layer "F.SilkS")
 		(effects
@@
 		)
 	)
+	(gr_text "TEMP"
+		(at 222.82 158.72 0)
+		(layer "F.SilkS")
+		(effects
+			(font
+				(size 0.5 0.5)
+				(thickness 0.125)
+			)
+			(justify left bottom)
+		)
+	)
 	(gr_text "SCK_ADC_EXT"
 		(at 196.42 149.72 0)
@@
 		)
 	)
+	(gr_text "+VCC"
+		(at 268.42 115.92 0)
+		(layer "F.SilkS")
+		(effects
+			(font
+				(size 0.5 0.5)
+				(thickness 0.125)
+			)
+			(justify left bottom)
+		)
+	)
+	(gr_text "RED"
+		(at 241.82 161.92 0)
+		(layer "F.SilkS")
+		(effects
+			(font
+				(size 0.5 0.5)
+				(thickness 0.125)
+			)
+			(justify left bottom)
+		)
+	)
 	(gr_text "+3V3"
 		(at 229.12 111.52 0)
@@
 		)
 	)
+	(gr_text "H3"
+		(at 214.72 158.72 0)
+		(layer "F.SilkS")
+		(effects
+			(font
+				(size 0.5 0.5)
+				(thickness 0.125)
+			)
+			(justify left bottom)
+		)
+	)
 	(gr_text "+5V"
 		(at 196.42 144.92 0)
@@
 		)
 	)
+	(gr_text "GND"
+		(at 195.62 159.72 0)
+		(layer "F.SilkS")
+		(effects
+			(font
+				(size 0.5 0.5)
+				(thickness 0.125)
+			)
+			(justify left bottom)
+		)
+	)
 	(gr_text "CAN_P"
 		(at 191.62 111.22 0)
@@
 			)
 			(justify left bottom)
+		)
+	)
+	(gr_text "THERMISTOR"
+		(at 193.494434 164.568184 90)
+		(layer "F.SilkS")
+		(effects
+			(font
+				(size 0.5 0.5)
+				(thickness 0.125)
+			)
+			(justify left bottom)

Commit message: update 20240428_2
Parts:
- moved G*** 0.80 mm to (280.3, 130.5)
- moved G*** 0.76 mm to (280.6, 147.6)
Routing:
- net HALL_1_OUT: track 24.1 -> 23.2 mm
Other:
- board text added: "+3V3 ON"
- board text added: "+VDC"
- board text added: "+VDC ON"
- board text added: "PHASE 1"
- board text added: "PHASE 2"
- board text added: "PHASE 3"
- board text added: "RESET"
- board text removed: "+VCC"
Changed lines of the file:
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@@
 	(footprint "LOGO"
 		(layer "F.Cu")
-		(at 280.32 131.32)
+		(at 280.32 130.52)
 		(property "Reference" "G***"
 			(at 0 0 0)
@@
 	(footprint "LOGO"
 		(layer "F.Cu")
-		(at 280.32 148.32)
+		(at 280.62 147.62)
 		(property "Reference" "G***"
 			(at 0 0 0)
@@
 		)
 	)
+	(gr_text "+3V3 ON"
+		(at 250.62 122.62 0)
+		(layer "F.SilkS")
+		(effects
+			(font
+				(size 0.5 0.5)
+				(thickness 0.125)
+			)
+			(justify left bottom)
+		)
+	)
 	(gr_text "CAN"
 		(at 191.82 105.92 0)
@@
 		)
 	)
+	(gr_text "+VDC ON"
+		(at 277.82 109.72 0)
+		(layer "F.SilkS")
+		(effects
+			(font
+				(size 0.5 0.5)
+				(thickness 0.125)
+			)
+			(justify left bottom)
+		)
+	)
 	(gr_text "GND"
 		(at 210.12 160.32 0)
@@
 		)
 	)
+	(gr_text "RESET"
+		(at 201.52 131.32 0)
+		(layer "F.SilkS")
+		(effects
+			(font
+				(size 0.7 0.7)
+				(thickness 0.15)
+			)
+			(justify left bottom)
+		)
+	)
 	(gr_text "+3V3_COM"
 		(at 196.42 146.52 0)
@@
 		)
 	)
+	(gr_text "PHASE 3"
+		(at 276.92 151.22 0)
+		(layer "F.SilkS")
+		(effects
+			(font
+				(size 1 1)
+				(thickness 0.15)
+			)
+			(justify left bottom)
+		)
+	)
 	(gr_text "H2"
 		(at 217.12 158.72 0)
@@
 		)
 	)
-	(gr_text "+VCC"
+	(gr_text "+VDC"
 		(at 268.42 115.92 0)
 		(layer "F.SilkS")
@@
 		)
 	)
+	(gr_text "PHASE 2"
+		(at 276.92 134.32 0)
+		(layer "F.SilkS")
+		(effects
+			(font
+				(size 1 1)
+				(thickness 0.15)
+			)
+			(justify left bottom)
+		)
+	)
 	(gr_text "CAN_P"
 		(at 191.62 111.22 0)
@@
 		)
 	)
+	(gr_text "PHASE 1"
+		(at 277.22 117.42 0)
+		(layer "F.SilkS")
+		(effects
+			(font
+				(size 1 1)
+				(thickness 0.15)
+			)
+			(justify left bottom)
+		)
+	)
 	(gr_text "Not specified"
 		(at 468.895715 257.515 0)
@@
 	)
 	(segment
-		(start 226.088628 151.42)
+		(start 226.788628 152.12)
 		(end 230.288628 155.62)
 		(width 0.2)
@@
 	)
 	(segment
-		(start 235.82 155.62)
-		(end 237.32 157.12)
+		(start 230.288628 155.62)
+		(end 235.82 155.62)
 		(width 0.2)
 		(layer "B.Cu")
@@
 	)
 	(segment
-		(start 230.288628 155.62)
-		(end 235.82 155.62)
+		(start 216.22 146.62)
+		(end 217.52 146.62)
 		(width 0.2)
 		(layer "B.Cu")
@@
 	)
 	(segment
-		(start 216.22 146.62)
-		(end 218.022942 146.62)
+		(start 237.32 157.12)
+		(end 237.32 159.4945)
 		(width 0.2)
 		(layer "B.Cu")
@@
 	)
 	(segment
-		(start 222.822943 151.42)
-		(end 226.088628 151.42)
+		(start 223.02 152.12)
+		(end 226.788628 152.12)
 		(width 0.2)
 		(layer "B.Cu")
@@
 	)
 	(segment
-		(start 218.022942 146.62)
-		(end 222.822943 151.42)
+		(start 235.82 155.62)
+		(end 237.32 157.12)
 		(width 0.2)
 		(layer "B.Cu")
@@
 	)
 	(segment
-		(start 237.32 157.12)
-		(end 237.32 159.4945)
+		(start 217.52 146.62)
+		(end 223.02 152.12)
 		(width 0.2)
 		(layer "B.Cu")
@@
 	)
 	(segment
-		(start 216.509831 144.541203)
-		(end 222.988628 151.02)
+		(start 230.454314 155.22)
+		(end 238.02 155.22)
 		(width 0.2)
 		(layer "B.Cu")
@@
 	)
 	(segment
-		(start 238.02 155.22)
-		(end 239.92 157.12)
+		(start 216.509831 143.088)
+		(end 216.509831 144.709831)
 		(width 0.2)
 		(layer "B.Cu")
@@
 	)
 	(segment
-		(start 226.254314 151.02)
-		(end 230.454314 155.22)
+		(start 216.509831 144.709831)
+		(end 223.22 151.42)
 		(width 0.2)
 		(layer "B.Cu")
@@
 	)
 	(segment
-		(start 230.454314 155.22)
-		(end 238.02 155.22)
+		(start 223.22 151.42)
+		(end 226.654314 151.42)
 		(width 0.2)
 		(layer "B.Cu")
@@
 	)
 	(segment
-		(start 239.92 157.12)
-		(end 239.92 159.4945)
+		(start 238.02 155.22)
+		(end 239.92 157.12)
 		(width 0.2)
 		(layer "B.Cu")
@@
 	)
 	(segment
-		(start 216.509831 143.088)
-		(end 216.509831 144.541203)
+		(start 226.654314 151.42)
+		(end 230.454314 155.22)
 		(width 0.2)
 		(layer "B.Cu")
@@
 	)
 	(segment
-		(start 222.988628 151.02)
-		(end 226.254314 151.02)
+		(start 239.92 157.12)
+		(end 239.92 159.4945)
 		(width 0.2)
 		(layer "B.Cu")
@@
 	)
 	(segment
-		(start 242.62 149.22)
-		(end 243.62 148.22)
+		(start 240.37 150.237033)
+		(end 240.352967 150.22)
 		(width 0.2)
 		(layer "B.Cu")
@@
 	)
 	(segment
-		(start 242.62 150.237033)
-		(end 242.62 149.22)
+		(start 242.62 149.22)
+		(end 243.62 148.22)
 		(width 0.2)
 		(layer "B.Cu")
@@
 	)
 	(segment
-		(start 223.32 150.22)
-		(end 240.352967 150.22)
+		(start 242.62 150.237033)
+		(end 242.62 149.22)
 		(width 0.2)
 		(layer "B.Cu")
@@
 	)
 	(segment
-		(start 240.352967 150.22)
-		(end 240.37 150.237033)
+		(start 218.02 141.82)
+		(end 217.72 141.52)
 		(width 0.2)
 		(layer "B.Cu")
@@
 	)
 	(segment
-		(start 217.72 141.52)
-		(end 217.12 141.52)
+		(start 242.62 150.237033)
+		(end 242.62 150.22)
 		(width 0.2)
 		(layer "B.Cu")
@@
 	)
 	(segment
-		(start 242.62 150.237033)
-		(end 242.62 150.22)
+		(start 223.72 150.22)
+		(end 218.02 144.52)
 		(width 0.2)
 		(layer "B.Cu")
@@
 	)
 	(segment
-		(start 218.02 141.82)
-		(end 217.72 141.52)
+		(start 243.62 148.22)
+		(end 247.22 148.22)
 		(width 0.2)
 		(layer "B.Cu")
@@
 	)
 	(segment
-		(start 243.62 148.22)
-		(end 247.22 148.22)
+		(start 217.72 141.52)
+		(end 217.12 141.52)
 		(width 0.2)
 		(layer "B.Cu")
@@
 	)
 	(segment
-		(start 223.32 150.22)
-		(end 218.02 144.92)
+		(start 240.352967 150.22)
+		(end 223.72 150.22)
 		(width 0.2)
 		(layer "B.Cu")
@@
 	)
 	(segment
-		(start 218.02 144.92)
+		(start 218.02 144.52)
 		(end 218.02 141.82)
 		(width 0.2)
@@
 	)
 	(segment
-		(start 241.72 156.92)
-		(end 239.62 154.82)
+		(start 223.62 150.82)
+		(end 217.12 144.32)
 		(width 0.2)
 		(layer "B.Cu")
@@
 	)
 	(segment
-		(start 217.12 142.52)
-		(end 215.92 141.32)
+		(start 241.72 159.52)
+		(end 241.72 156.92)
 		(width 0.2)
 		(layer "B.Cu")
@@
 	)
 	(segment
-		(start 226.42 150.62)
-		(end 223.154314 150.62)
+		(start 230.62 154.82)
+		(end 226.62 150.82)
 		(width 0.2)
 		(layer "B.Cu")
@@
 	)
 	(segment
-		(start 217.12 144.585686)
-		(end 217.12 142.52)
+		(start 226.62 150.82)
+		(end 223.62 150.82)
 		(width 0.2)
 		(layer "B.Cu")
@@
 	)
 	(segment
-		(start 223.154314 150.62)
-		(end 217.12 144.585686)
+		(start 217.12 142.52)
+		(end 215.92 141.32)
 		(width 0.2)
 		(layer "B.Cu")
@@
 	)
 	(segment
-		(start 230.62 154.82)
-		(end 226.42 150.62)
+		(start 241.72 156.92)
+		(end 239.62 154.82)
 		(width 0.2)
 		(layer "B.Cu")
@@
 	)
 	(segment
-		(start 241.72 159.52)
-		(end 241.72 156.92)
+		(start 217.12 144.32)
+		(end 217.12 142.52)
 		(width 0.2)
 		(layer "B.Cu")
@@
 	)
 	(segment
-		(start 215.12 137.42)
-		(end 215.12 141.52)
+		(start 215.62 146.868529)
+		(end 215.971471 147.22)
 		(width 0.2)
 		(layer "B.Cu")
@@
 	)
 	(segment
-		(start 215.62 142.02)
-		(end 215.62 146.868529)
+		(start 215.971471 147.22)
+		(end 216.32 147.22)
 		(width 0.2)
 		(layer "B.Cu")
@@
 	)
 	(segment
-		(start 215.12 141.52)
-		(end 215.62 142.02)
+		(start 215.12 137.42)
+		(end 215.12 141.52)
 		(width 0.2)
 		(layer "B.Cu")
@@
 	)
 	(segment
-		(start 215.971471 147.22)
-		(end 217.82 147.22)
+		(start 218.92 149.82)
+		(end 218.92 153.22)
 		(width 0.2)
 		(layer "B.Cu")
@@
 	)
 	(segment
-		(start 218.92 148.32)
-		(end 218.92 153.22)
+		(start 215.12 141.52)
+		(end 215.62 142.02)
 		(width 0.2)
 		(layer "B.Cu")
@@
 	)
 	(segment
-		(start 215.62 146.868529)
-		(end 215.971471 147.22)
+		(start 215.62 142.02)
+		(end 215.62 146.868529)
 		(width 0.2)
 		(layer "B.Cu")
@@
 	)
 	(segment
-		(start 217.82 147.22)
-		(end 218.92 148.32)
+		(start 216.32 147.22)
+		(end 218.92 149.82)
 		(width 0.2)
 		(layer "B.Cu")
@@
 	)
 	(segment
-		(start 218.82 145.02)
+		(start 218.82 144.52)
 		(end 218.82 138.82)
 		(width 0.2)
@@
 	)
 	(segment
-		(start 223.02 149.22)
-		(end 218.82 145.02)
+		(start 235.62 149.22)
+		(end 223.52 149.22)
 		(width 0.2)
 		(layer "B.Cu")
@@
 	)
 	(segment
-		(start 235.62 149.22)
-		(end 223.02 149.22)
+		(start 223.52 149.22)
+		(end 218.82 144.52)
 		(width 0.2)
 		(layer "B.Cu")
