File: Projects/Client Name/DF_ESC/Design/rev01/rev01_1/DF_ESC_rev01_1/MCU.kicad_sch (KiCad schematic)
At the start: 37 parts, among them J2 HX25003-8AWB, J3 S6B-XH-SM4-TB(LF)(SN), J4 XH-3AWB, SW1 SW_DIP_x01, U3 STM32F405RGTx, Y1 Crystal_Small

Commit message: Update 20240416
Lesson 16 finished
Parts:
- added R64: 2k2, Resistor_SMD:R_0603_1608Metric_Pad0.98x0.95mm_HandSolder, symbol Device:R
- D7: footprint PESD3V3U1UA:SOD-323_L1.7-W1.3-LS2.5-RD -> Diode_SMD:D_SOD-323_HandSoldering
- D9: footprint Diode_SMD:D_SOD-323 -> Diode_SMD:D_SOD-323_HandSoldering
Connections:
- net GND: now also R64.2; no longer SW1.1
- new net: R64.1, SW1.1
Changed lines of the file:
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@@
 	(wire
 		(pts
-			(xy 114.3 48.26) (xy 114.3 55.88)
-		)
-		(stroke
-			(width 0)
-			(type default)
-		)
-	)
-	(wire
-		(pts
 			(xy 96.52 49.53) (xy 96.52 46.99)
 		)
@@
 	(wire
 		(pts
+			(xy 111.76 48.26) (xy 111.76 49.53)
+		)
+		(stroke
+			(width 0)
+			(type default)
+		)
+	)
+	(wire
+		(pts
 			(xy 143.51 128.27) (xy 143.51 130.81)
 		)
@@
 	(wire
 		(pts
+			(xy 111.76 57.15) (xy 111.76 58.42)
+		)
+		(stroke
+			(width 0)
+			(type default)
+		)
+	)
+	(wire
+		(pts
 			(xy 29.21 186.69) (xy 43.18 186.69)
 		)
@@
 	(wire
 		(pts
+			(xy 114.3 48.26) (xy 111.76 48.26)
+		)
+		(stroke
+			(width 0)
+			(type default)
+		)
+	)
+	(wire
+		(pts
 			(xy 245.11 132.08) (xy 250.19 132.08)
 		)
@@
 	)
 	(symbol
+		(lib_id "Device:R")
+		(at 111.76 53.34 0)
+		(unit 1)
+		(exclude_from_sim no)
+		(in_bom yes)
+		(on_board yes)
+		(dnp no)
+		(property "Reference" "R64"
+			(at 113.538 50.8 0)
+			(effects
+				(font
+					(size 1.27 1.27)
+				)
+				(justify left)
+			)
+		)
+		(property "Value" "2k2"
+			(at 113.538 56.896 0)
+			(effects
+				(font
+					(size 1.27 1.27)
+				)
+				(justify left)
+			)
+		)
+		(property "Footprint" "Resistor_SMD:R_0603_1608Metric_Pad0.98x0.95mm_HandSolder"
+			(at 109.982 53.34 90)
+			(effects
+				(font
+					(size 1.27 1.27)
+				)
+				(hide yes)
+			)
+		)
+		(property "Datasheet" "~"
+			(at 111.76 53.34 0)
+			(effects
+				(font
+					(size 1.27 1.27)
+				)
+				(hide yes)
+			)
+		)
+		(property "Description" "Resistor"
+			(at 111.76 53.34 0)
+			(effects
+				(font
+					(size 1.27 1.27)
+				)
+				(hide yes)
+			)
+		)
+		(pin "2"
+		)
+		(pin "1"
+		)
+		(instances
+			(project "DF_ESC_rev01_1"
+				(path "/e63e39d7-6ac0-4ffd-8aa3-1841a4541b55/138932fe-f685-46a1-bb06-1768136a532b"
+					(reference "R64")
+					(unit 1)
+				)
+			)
+		)
+	)
+	(symbol
 		(lib_id "Device:C")
 		(at 143.51 134.62 0)
@@
 			)
 		)
-		(property "Footprint" "Diode_SMD:D_SOD-323"
+		(property "Footprint" "Diode_SMD:D_SOD-323_HandSoldering"
 			(at 91.44 176.53 0)
 			(effects
@@
 			)
 		)
-		(property "Footprint" "PESD3V3U1UA:SOD-323_L1.7-W1.3-LS2.5-RD"
+		(property "Footprint" "Diode_SMD:D_SOD-323_HandSoldering"
 			(at 59.69 175.26 0)
 			(effects
@@
 		)
 		(property "Value" "SW_DIP_x01"
-			(at 121.92 53.34 0)
+			(at 125.222 52.578 0)
 			(effects
 				(font
@@
 	(symbol
 		(lib_id "power:GND")
-		(at 114.3 55.88 0)
+		(at 111.76 58.42 0)
 		(unit 1)
 		(exclude_from_sim no)
@@
 		(fields_autoplaced yes)
 		(property "Reference" "#PWR027"
-			(at 114.3 62.23 0)
+			(at 111.76 64.77 0)
 			(effects
 				(font
@@
 		)
 		(property "Value" "GND"
-			(at 114.3 60.96 0)
+			(at 111.76 63.5 0)
 			(effects
 				(font
@@
 		)
 		(property "Footprint" ""
-			(at 114.3 55.88 0)
+			(at 111.76 58.42 0)
 			(effects
 				(font
@@
 		)
 		(property "Datasheet" ""
-			(at 114.3 55.88 0)
+			(at 111.76 58.42 0)
 			(effects
 				(font
@@
 		)
 		(property "Description" ""
-			(at 114.3 55.88 0)
+			(at 111.76 58.42 0)
 			(effects
 				(font

Commit message: update 20240427
Mejora de layout cero errores, solo falta añadir algunas reseñas en el silkscreen
Parts:
- J3: footprint DF_ESC_Footprint_Library_Casa:CONN-SMD_S6B-XH-SM4-TB-LF-SN -> DF_ESC_Footprint_Library:CONN-SMD_S6B-XH-SM4-TB-LF-SN
- J4: footprint DF_ESC_Footprint_Library_Casa:CONN-SMD_XH-3AWB -> DF_ESC_Footprint_Library:CONN-SMD_XH-3AWB
- SW1: footprint DF_ESC_Footprint_Library_Casa:SW-SMD_4P-L5.2-W5.2-P3.70-LS6.4 -> DF_ESC_Footprint_Library:SW-SMD_4P-L5.2-W5.2-P3.70-LS6.4
- Y1: footprint DF_ESC_Footprint_Library_Casa:CRYSTAL-SMD_L5.0-W3.2 -> DF_ESC_Footprint_Library:CRYSTAL-SMD_L5.0-W3.2
Changed lines of the file:
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@@
 			)
 		)
-		(property "Footprint" "DF_ESC_Footprint_Library_Casa:CONN-SMD_S6B-XH-SM4-TB-LF-SN"
+		(property "Footprint" "DF_ESC_Footprint_Library:CONN-SMD_S6B-XH-SM4-TB-LF-SN"
 			(at 265.43 113.03 0)
 			(effects
@@
 			)
 		)
-		(property "Footprint" "DF_ESC_Footprint_Library_Casa:CRYSTAL-SMD_L5.0-W3.2"
+		(property "Footprint" "DF_ESC_Footprint_Library:CRYSTAL-SMD_L5.0-W3.2"
 			(at 93.98 76.2 0)
 			(effects
@@
 			)
 		)
-		(property "Footprint" "DF_ESC_Footprint_Library_Casa:CONN-SMD_XH-3AWB"
+		(property "Footprint" "DF_ESC_Footprint_Library:CONN-SMD_XH-3AWB"
 			(at 270.51 142.24 0)
 			(effects
@@
 			)
 		)
-		(property "Footprint" "DF_ESC_Footprint_Library_Casa:SW-SMD_4P-L5.2-W5.2-P3.70-LS6.4"
+		(property "Footprint" "DF_ESC_Footprint_Library:SW-SMD_4P-L5.2-W5.2-P3.70-LS6.4"
 			(at 121.92 48.26 0)
 			(effects
