File: Projects/Client Name/DF_ESC/Design/rev01/rev01_1/DF_ESC_rev01_1/MOSFET DRIVER.kicad_sch (KiCad schematic)
At the start: 40 parts, among them U4 DRV8302DCAR

Commit message: Update 2024-03-13_2
Version final para posicionar PCB
Parts:
- U4: footprint footprint:HTSSOP-56_L14.0-W6.1-P0.50-LS8.1-BL-EP -> DF_ESC_Footprint_Library:HTSSOP-56_L14.0-W6.1-P0.50-LS8.1-BL-EP
Changed lines of the file:
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@@
 			)
 		)
-		(property "Footprint" "footprint:HTSSOP-56_L14.0-W6.1-P0.50-LS8.1-BL-EP"
+		(property "Footprint" "DF_ESC_Footprint_Library:HTSSOP-56_L14.0-W6.1-P0.50-LS8.1-BL-EP"
 			(at 130.81 66.04 0)
 			(effects

Commit message: Update 20240416
Lesson 16 finished
Parts:
- C41, C43, C45: footprint Capacitor_SMD:C_0603_1608Metric_Pad1.08x0.95mm_HandSolder -> Capacitor_SMD:C_1210_3225Metric
Changed lines of the file:
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@@
 			)
 		)
-		(property "Footprint" "Capacitor_SMD:C_0603_1608Metric_Pad1.08x0.95mm_HandSolder"
+		(property "Footprint" "Capacitor_SMD:C_1210_3225Metric"
 			(at 210.5152 99.06 0)
 			(effects
@@
 			)
 		)
-		(property "Footprint" "Capacitor_SMD:C_0603_1608Metric_Pad1.08x0.95mm_HandSolder"
+		(property "Footprint" "Capacitor_SMD:C_1210_3225Metric"
 			(at 215.5952 99.06 0)
 			(effects
@@
 			)
 		)
-		(property "Footprint" "Capacitor_SMD:C_0603_1608Metric_Pad1.08x0.95mm_HandSolder"
+		(property "Footprint" "Capacitor_SMD:C_1210_3225Metric"
 			(at 205.4352 99.06 0)
 			(effects

Commit message: update 20240427
Mejora de layout cero errores, solo falta añadir algunas reseñas en el silkscreen
Parts:
- L1: footprint DF_ESC_Footprint_Library_Casa:IND-SMD_L7.8-W7.8_SDR0805 -> DF_ESC_Footprint_Library:IND-SMD_L7.8-W7.8_SDR0805
Changed lines of the file:
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@@
 			)
 		)
-		(property "Footprint" "DF_ESC_Footprint_Library_Casa:IND-SMD_L7.8-W7.8_SDR0805"
+		(property "Footprint" "DF_ESC_Footprint_Library:IND-SMD_L7.8-W7.8_SDR0805"
 			(at 199.39 86.36 0)
 			(effects
